File: Relay.sch (KiCad schematic (older format))
At the start: 0 parts

Commit message: Understanding the Relay Module
Parts:
- added D?: LED, symbol LED
- added D?: DIODE, symbol DIODE
- added K?: RELAY_SPDT, symbol RELAY_SPDT
- added Q?: NPN, symbol NPN
- added R? (x6): R, symbol R
- added U?: PHTRANS, symbol PHTRANS
Connections:
- net DIN+: now also U?.1
- net DIN-: now also R?.1
- new net: D?.2 (K), K?.2 (COIL_+), R?.1, R?.2, U?.5
- new net: D?.1 (A), K?.5 (COIL_-), Q?.3 (C)
- new net: R?.2, U?.2
- new net: D?.1 (A), R?.1, U?.4
- new net: R?.1, U?.6
- new net: Q?.2 (B), R?.2
- new net: Q?.1 (E), R?.2
- new net: D?.2 (K), R?.2
- new net +12V: R?.2
- new net COM: K?.1 (COM)
- new net GND: R?.1, R?.1
- new net NC: K?.4 (NC)
- new net NO: K?.3 (NO)
Changed lines of the file:
@@
 Comment4 ""
 $EndDescr
-Text HLabel 2400 3100 0    60   Input ~ 0
+Text HLabel 4200 3100 0    60   Input ~ 0
 DIN+
-Text HLabel 2400 3300 0    60   Output ~ 0
+Text HLabel 4200 3450 0    60   Output ~ 0
 DIN-
-Text HLabel 8000 2950 0    60   Input ~ 0
-Relay+
-Text HLabel 8000 3200 0    60   Output ~ 0
-Relay-
+Text HLabel 10500 2100 2    60   BiDi ~ 0
+NC
+Text HLabel 10500 2300 2    60   BiDi ~ 0
+NO
+$Comp
+L RELAY_SPDT K?
+U 1 1 52F1DB37
+P 9800 2350
+F 0 "K?" H 9800 2750 70  0000 C CNN
+F 1 "RELAY_SPDT" H 9800 2000 70  0000 C CNN
+F 2 "" H 9800 2550 60  0000 C CNN
+F 3 "" H 9800 2550 60  0000 C CNN
+	1    9800 2350
+	1    0    0    -1
+$EndComp
+$Comp
+L PHTRANS U?
+U 1 1 52F1DB4B
+P 6300 3300
+F 0 "U?" H 6250 3650 70  0000 C CNN
+F 1 "PHTRANS" H 6250 2950 70  0000 C CNN
+F 2 "" H 6300 3300 60  0000 C CNN
+F 3 "" H 6300 3300 60  0000 C CNN
+	1    6300 3300
+	1    0    0    -1
+$EndComp
+$Comp
+L R R?
+U 1 1 52F1DB5F
+P 7650 3500
+F 0 "R?" V 7730 3500 40  0000 C CNN
+F 1 "R" V 7657 3501 40  0000 C CNN
+F 2 "" V 7580 3500 30  0000 C CNN
+F 3 "" H 7650 3500 30  0000 C CNN
+	1    7650 3500
+	0    -1   -1   0
+$EndComp
+$Comp
+L NPN Q?
+U 1 1 52F1DB73
+P 8950 3500
+F 0 "Q?" H 8950 3350 50  0000 R CNN
+F 1 "NPN" H 8950 3650 50  0000 R CNN
+F 2 "" H 8950 3500 60  0000 C CNN
+F 3 "" H 8950 3500 60  0000 C CNN
+	1    8950 3500
+	1    0    0    -1
+$EndComp
+$Comp
+L LED D?
+U 1 1 52F1DB87
+P 7100 4000
+F 0 "D?" H 7100 4100 50  0000 C CNN
+F 1 "LED" H 7100 3900 50  0000 C CNN
+F 2 "" H 7100 4000 60  0000 C CNN
+F 3 "" H 7100 4000 60  0000 C CNN
+	1    7100 4000
+	0    1    1    0
+$EndComp
+Text HLabel 10500 1650 2    60   BiDi ~ 0
+COM
+Wire Wire Line
+	10500 1650 8600 1650
+Wire Wire Line
+	8600 1650 8600 2200
+Wire Wire Line
+	8600 2200 9400 2200
+Wire Wire Line
+	10500 2100 10200 2100
+Wire Wire Line
+	10500 2300 10200 2300
+Wire Wire Line
+	7900 3500 8750 3500
+Wire Wire Line
+	7900 2100 7900 3300
+Wire Wire Line
+	6850 3500 7400 3500
+$Comp
+L R R?
+U 1 1 52F1DDD5
+P 9050 4250
+F 0 "R?" V 9130 4250 40  0000 C CNN
+F 1 "R" V 9057 4251 40  0000 C CNN
+F 2 "" V 8980 4250 30  0000 C CNN
+F 3 "" H 9050 4250 30  0000 C CNN
+	1    9050 4250
+	-1   0    0    1
+$EndComp
+Wire Wire Line
+	9050 3700 9050 4000
+$Comp
+L GND #PWR?
+U 1 1 52F1DE0A
+P 9050 4750
+F 0 "#PWR?" H 9050 4750 30  0001 C CNN
+F 1 "GND" H 9050 4680 30  0001 C CNN
+F 2 "" H 9050 4750 60  0000 C CNN
+F 3 "" H 9050 4750 60  0000 C CNN
+	1    9050 4750
+	1    0    0    -1
+$EndComp
+Wire Wire Line
+	9050 4750 9050 4500
+$Comp
+L R R?
+U 1 1 52F1DE43
+P 7100 4600
+F 0 "R?" V 7180 4600 40  0000 C CNN
+F 1 "R" V 7107 4601 40  0000 C CNN
+F 2 "" V 7030 4600 30  0000 C CNN
+F 3 "" H 7100 4600 30  0000 C CNN
+	1    7100 4600
+	-1   0    0    1
+$EndComp
+$Comp
+L GND #PWR?
+U 1 1 52F1DE4E
+P 7100 5100
+F 0 "#PWR?" H 7100 5100 30  0001 C CNN
+F 1 "GND" H 7100 5030 30  0001 C CNN
+F 2 "" H 7100 5100 60  0000 C CNN
+F 3 "" H 7100 5100 60  0000 C CNN
+	1    7100 5100
+	1    0    0    -1
+$EndComp
+Wire Wire Line
+	7100 5100 7100 4850
+Wire Wire Line
+	7100 4350 7100 4200
+Wire Wire Line
+	7100 3800 7100 3500
+Connection ~ 7100 3500
+$Comp
+L R R?
+U 1 1 52F1DE8A
+P 7900 1850
+F 0 "R?" V 7980 1850 40  0000 C CNN
+F 1 "R" V 7907 1851 40  0000 C CNN
+F 2 "" V 7830 1850 30  0000 C CNN
+F 3 "" H 7900 1850 30  0000 C CNN
+	1    7900 1850
+	-1   0    0    1
+$EndComp
+$Comp
+L +12V #PWR?
+U 1 1 52F1DE97
+P 7900 1400
+F 0 "#PWR?" H 7900 1350 20  0001 C CNN
+F 1 "+12V" H 7900 1500 30  0000 C CNN
+F 2 "" H 7900 1400 60  0000 C CNN
+F 3 "" H 7900 1400 60  0000 C CNN
+	1    7900 1400
+	1    0    0    -1
+$EndComp
+Wire Wire Line
+	7900 1400 7900 1600
+Wire Wire Line
+	7900 3300 6850 3300
+$Comp
+L R R?
+U 1 1 52F1DED1
+P 7300 3100
+F 0 "R?" V 7380 3100 40  0000 C CNN
+F 1 "R" V 7307 3101 40  0000 C CNN
+F 2 "" V 7230 3100 30  0000 C CNN
+F 3 "" H 7300 3100 30  0000 C CNN
+	1    7300 3100
+	0    -1   -1   0
+$EndComp
+Wire Wire Line
+	6850 3100 7050 3100
+Wire Wire Line
+	7550 3100 7900 3100
+Connection ~ 7900 3100
+$Comp
+L R R?
+U 1 1 52F1DF0A
+P 5250 3450
+F 0 "R?" V 5330 3450 40  0000 C CNN
+F 1 "R" V 5257 3451 40  0000 C CNN
+F 2 "" V 5180 3450 30  0000 C CNN
+F 3 "" H 5250 3450 30  0000 C CNN
+	1    5250 3450
+	0    -1   -1   0
+$EndComp
+Wire Wire Line
+	5500 3450 5750 3450
+Wire Wire Line
+	4200 3450 5000 3450
+Wire Wire Line
+	4200 3100 5750 3100
+$Comp
+L DIODE D?
+U 1 1 52F1DF69
+P 8450 2750
+F 0 "D?" H 8450 2850 40  0000 C CNN
+F 1 "DIODE" H 8450 2650 40  0000 C CNN
+F 2 "" H 8450 2750 60  0000 C CNN
+F 3 "" H 8450 2750 60  0000 C CNN
+	1    8450 2750
+	0    -1   -1   0
+$EndComp
+Wire Wire Line
+	9400 2500 9050 2500
+Wire Wire Line
+	9050 2500 9050 3300
+Wire Wire Line
+	9400 2400 7900 2400
+Connection ~ 7900 2400
+Wire Wire Line
+	8450 2400 8450 2550
+Connection ~ 8450 2400
+Wire Wire Line
+	8450 2950 8450 3100
+Wire Wire Line
+	8450 3100 9050 3100
+Connection ~ 9050 3100
 $EndSCHEMATC
