File: Relay.sch (KiCad schematic (older format))
At the start: 11 parts

Commit message: Understanding the Arduino Module
Connections:
- net labels added: RELAY+, RELAY-, RELAY_COM, RELAY_NC, RELAY_NO
- net labels removed: COM, DIN+, DIN-, NC, NO
Changed lines of the file:
@@
 LIBS:valves
 LIBS:MyComponents
+LIBS:arduino_shieldsNCL
 LIBS:BenchBuddy-cache
 EELAYER 24 0
@@
 $Descr A4 11693 8268
 encoding utf-8
-Sheet 9 9
+Sheet 7 9
 Title ""
 Date ""
@@
 $EndDescr
 Text HLabel 4200 3100 0    60   Input ~ 0
-DIN+
+RELAY+
 Text HLabel 4200 3450 0    60   Output ~ 0
-DIN-
+RELAY-
 Text HLabel 10500 2100 2    60   BiDi ~ 0
-NC
+RELAY_NC
 Text HLabel 10500 2300 2    60   BiDi ~ 0
-NO
+RELAY_NO
 $Comp
 L RELAY_SPDT K?
@@
 $EndComp
 Text HLabel 10500 1650 2    60   BiDi ~ 0
-COM
+RELAY_COM
 Wire Wire Line
 	10500 1650 8600 1650

Commit message: Associating and Placing the Relay Module
Parts:
- removed R?: R, symbol R
- removed U?: PHTRANS, symbol PHTRANS
- added R38: 0, symbol R
- added U9: LTV-816S, symbol OPTO-TRANSISTOR4
- D2: renamed from D?; MFG Part Number (none) -> LG Q971-KN-1
- D3: renamed from D?; value DIODE -> B130-13-F; MFG Name (none) -> Diodes Inc; MFG Part Number (none) -> B130-13-F
- K1: renamed from K?; value RELAY_SPDT -> 1461069-5
- Q1: renamed from Q?; value NPN -> 2N3904; MFG Name (none) -> Diodes Inc; MFG Part Number (none) -> MMBT3904-7-F
- R34: renamed from R?; value R -> 500
- R35: renamed from R?; value R -> 200
- R36: renamed from R?; value R -> 100
- R37, R39: renamed from R?; value R -> 0
Other:
- moved on the sheet: D2, D3, Q1, R34, R35, R36, R37, R39

Commit message: Merge CE BenchBudEE commit 00937c39d96b9ebb1b0292c11cc231788ab24edd
Parts:
- removed D2: LED, symbol LED
- removed D3: B130-13-F, symbol DIODE
- removed K1: 1461069-5, symbol RELAY_SPDT
- removed R34: 500, symbol R
- removed R35: 200, symbol R
- removed R36: 100, symbol R
- removed R37, R38, R39: 0, symbol R
- removed U9: LTV-816S, symbol OPTO-TRANSISTOR4
- added D1: LG Q971-KN-1, ~, symbol LED
- added D2: B130-13-F, ~, symbol DIODE
- added K1: 1461069-5, ~, symbol SPDT
- added R1: 500, ~, symbol R
- added R2: 200, ~, symbol R
- added R3, R5, R6: 0, ~, symbol R
- added R4: 100, ~, symbol R
- added U1: LTV-816S, symbol OPTO-TRANSISTOR4
- Q1: footprint (none) -> ~
Connections:
- net labels added: +12P
- net labels removed: +12V
- wire segments 26 -> 31

Commit message: Layout Work Session 4
Connections:
- net GND renamed GND_RELAY
Changed lines of the file:
@@
-	1    0    0    -1
-$EndComp
-$Comp
-L GND #PWR019
-U 1 1 523B9FB4
-P 8800 5650
-F 0 "#PWR019" H 8800 5650 30  0001 C CNN
-F 1 "GND" H 8800 5580 30  0001 C CNN
-F 2 "" H 8800 5650 60  0000 C CNN
-F 3 "" H 8800 5650 60  0000 C CNN
-	1    8800 5650
 	1    0    0    -1
 $EndComp
@@
 $EndComp
 $Comp
-L +12P #PWR020
+L +12P #PWR019
 U 1 1 523BA00D
 P 6450 1450
-F 0 "#PWR020" H 6450 1420 30  0001 C CNN
+F 0 "#PWR019" H 6450 1420 30  0001 C CNN
 F 1 "+12P" H 6450 1550 30  0000 C CNN
 F 2 "" H 6450 1450 60  0000 C CNN
@@
 	8100 1550 6450 1550
 Connection ~ 6450 1550
+$Comp
+L GND_RELAY #PWR020
+U 1 1 5313E55E
+P 8800 5650
+F 0 "#PWR020" H 8800 5650 30  0001 C CNN
+F 1 "GND_RELAY" H 8800 5580 30  0000 C CNN
+F 2 "" H 8800 5650 60  0000 C CNN
+F 3 "" H 8800 5650 60  0000 C CNN
+	1    8800 5650
+	1    0    0    -1
+$EndComp
 $EndSCHEMATC
