File: Power_Adjustment_Monitor.sch (KiCad schematic (older format))
At the start: 0 parts

Commit message: Understanding the Power Control, Conditioning and Monitoring Module
Parts:
- added JP? (x3): JUMPER, symbol JUMPER
- added R? (x8): R, symbol R
- added R? (x2): RVAR, symbol RVAR
- added U? (x2): LM317, symbol LM317_SOT223
- added U? (x2): 7805, symbol 7805
- added U? (x2): LM324, symbol LM324
Connections:
- net labels added: +12V, +3.3V, +5V, -12V, 3V3_MON, 5V_MON, AGND, FE_V+, FE_V-, GND, V+_ADJ, V+_ADJ_MON, V+_CURR_MON, V+_MON, V-_ADJ, V-_ADJ_MON, V-_CURR_MON, V-_MON
- wire segments 0 -> 98

Commit message: Associating and Placing the Relay Module
Parts:
- gave numbers to parts that had none: 18
Connections:
- wire segments 98 -> 77

Commit message: Merge CE BenchBudEE commit 00937c39d96b9ebb1b0292c11cc231788ab24edd
Parts:
- removed JP2, JP3: JUMPER, symbol JUMPER
- removed R24: RVAR, symbol RVAR
- removed U4, U7: LM317, symbol LM317_SOT223
- removed U5, U6: 7805, symbol 7805
- removed U8: LM324, symbol LM324
- added C13, C14, C15, C16, C17, C18, C19, C20, C21, C22, C23, C24: C, symbol C
- added D1, D10, D11, D12, D6, D7, D8, D9: MMBD914-7-F, symbol DIODE
- added R24: R, symbol R
- added R54: 5K, symbol RVAR
- added R55: 715, symbol R
- added U4, U7: LM317T, TO-220, symbol LM317T
- added U5, U6: LM337T, TO-220, symbol LM337T
- R26: value R -> 715
- R27: value RVAR -> 5K
Connections:
- net labels removed: V+_CURR_MON, V+_MON, V-_CURR_MON, V-_MON
- wire segments 77 -> 112
Other:
- note added: "+1.5v to +10v Output"
- note added: "+10v Output"
- note added: "-1.5v to -10v Output"
- note added: "-10v Output"
- moved on the sheet: JP1, R30, R31, R32, R33
