File: Arduino.sch (KiCad schematic (older format))
At the start: 21 parts

Commit message: Associating and Placing the Current/Fan Driver Module
Parts:
- added R52, R53: R, symbol R
Connections:
- net labels added: ~LDAC, ~SHDN
- wire segments 45 -> 49
Changed lines of the file:
@@
 Wire Wire Line
 	3400 3950 3750 3950
+$Comp
+L R R53
+U 1 1 530AA9BD
+P 7050 4750
+F 0 "R53" V 7050 4850 40  0000 C CNN
+F 1 "R" V 7057 4751 40  0000 C CNN
+F 2 "" V 6980 4750 30  0000 C CNN
+F 3 "" H 7050 4750 30  0000 C CNN
+	1    7050 4750
+	0    -1   -1   0
+$EndComp
+$Comp
+L R R52
+U 1 1 530AA9C8
+P 7050 4650
+F 0 "R52" V 7050 4750 40  0000 C CNN
+F 1 "R" V 7057 4651 40  0000 C CNN
+F 2 "" V 6980 4650 30  0000 C CNN
+F 3 "" H 7050 4650 30  0000 C CNN
+	1    7050 4650
+	0    -1   -1   0
+$EndComp
+Wire Wire Line
+	6800 4650 6450 4650
+Wire Wire Line
+	6800 4750 6450 4750
+Wire Wire Line
+	7300 4650 7600 4650
+Wire Wire Line
+	7300 4750 7600 4750
+Text HLabel 7600 4650 2    60   Output ~ 0
+~LDAC
+Text HLabel 7600 4750 2    60   Output ~ 0
+~SHDN
 $EndSCHEMATC

Commit message: Merge CE BenchBudEE commit 00937c39d96b9ebb1b0292c11cc231788ab24edd
Parts:
- removed Arduino1: ARDUINO_SHIELD, symbol ARDUINO_SHIELD
- removed R1, R10, R11, R12, R13, R14, R15, R2, R3, R4, R45, R49, R5, R52, R53, R6, R7, R8, R9: R, symbol R
- added ARD1: ARDUINOPINS, ~, symbol ARDUINOPINS
- added R26, R27, R28, R29, R30, R31, R32, R33, R34, R35, R36, R37, R38, R39, R40, R41, R42, R43, R47: R, ~, symbol R
- R46, R50, R51: footprint (none) -> ~
Other:
- note added: "The signal Digital5 was skipped so the pin numbers for all the following pins are off by one."

Commit message: Layout Work Session 2
Parts:
- removed ARD1: ARDUINOPINS, ~, symbol ARDUINOPINS
- added ARD1: ARDUINOPINS, symbol ARDUINO_SHIELD
Other:
- moved on the sheet: R26, R27, R28, R29, R30, R31, R32, R33, R34, R35, R36, R37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

Commit message: Layout Work Session 6
Pulled from CE
Parts:
- removed ARD1: ARDUINOPINS, symbol ARDUINO_SHIELD
- added ARD1: ARDUINOPINS, ~, symbol ARDUINOPINS
Other:
- moved on the sheet: R26, R27, R28, R29, R30, R31, R32, R33, R34, R35, R36, R37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
