File: BenchBuddy.kicad_pcb (KiCad board)
At the start: 4 copper layers, 165.1 x 63.5 mm, 127 parts, among them K1 1461069-5, P1 24 Pin MiniFit JR, P2 CONN_3X2, P3 CONN_2, P4 12 Pin Terminal Block, P5 3 Pin TB, Q1 2N3904, Q2 DMN65D8L-7, Q3 AOD476, Q4 AOD476, SW1 Power Switch, U1 LTV-816S, U11 LM317T, U2 MCP3901, U3 LMT84, U4 OPA4170, U5 MCP4801, U6 LM337T, U7 AP5726, U8 LM337T, U9 LM317T

Commit message: Layout Work Session 3
Parts:
- added HEATSINK_V8508H: VAL**, BenchBudEE:HEATSINK_V8508H, F.Cu at (241.0, 108.5)
- added HEATSINK_V8508H: VAL**, BenchBudEE:HEATSINK_V8508H, F.Cu at (259.6, 108.5)
- moved R19 43.6 mm to (193.6, 98.9)
- moved R20 43.6 mm to (209.3, 98.9)
- moved U11 40.3 mm to (259.6, 105.2), turned to 0 degrees
- moved U6 38.6 mm to (241.0, 105.1), turned to 0 degrees
- moved U2 15.6 mm to (245.0, 116.0), turned to 180 degrees
- moved U8 14.6 mm to (280.3, 106.0), turned to 0 degrees
- moved P2 8.17 mm to (263.4, 116.0)
- moved U4 6.89 mm to (278.8, 116.0)
- moved C1 1.70 mm to (214.2, 135.6)
- moved C7 1.70 mm to (209.4, 136.2)
- moved C8 1.70 mm to (211.6, 136.2)
- moved P3 1.70 mm to (205.4, 135.4)
- moved R26 1.70 mm to (201.9, 152.1)
- moved R27 1.70 mm to (204.5, 152.1)
- moved R28 1.70 mm to (206.9, 152.1)
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
Commit message: Layout Work Session 4
Parts:
- R17: moved to F.Cu
- moved R17 12.0 mm to (262.0, 134.9), turned to 180 degrees
- moved HEATSINK_V8508H 9.59 mm to (241.0, 98.9), turned to 0 degrees
- moved HEATSINK_V8508H 9.59 mm to (259.6, 98.9), turned to 0 degrees
- moved U7 8.59 mm to (255.5, 134.9)
- moved D4 0.89 mm to (290.3, 126.2)
- moved Q3 0.52 mm to (284.1, 126.5)
Connections:
- C10 pad 1: AGND -> GND_TC
- C11 pad 2: AGND -> GND_TC
- C12 pad 1: AGND -> GND_FAN
- C13 pad 2: GND -> GND_FAN
- C14 pad 2: AGND -> GND_TC
- C15 pad 1: AGND -> GND_TC
- C16 pad 2: AGND -> GND_PWR
- C17 pad 2: AGND -> GND_PWR
- C18 pad 2: AGND -> GND_PWR
- C19 pad 2: AGND -> GND_PWR
- C20 pad 2: AGND -> GND_TC
- C21 pad 1: AGND -> GND_TC
- C22 pad 2: AGND -> GND_PWR
- C23 pad 2: FE_V- -> GND_PWR
- C24 pad 2: AGND -> GND_TC
- C25 pad 2: AGND -> GND_TC
- C5 pad 2: GND -> GND_LED
- C6 pad 2: GND -> GND_LED
- C7 pad 1: AGND -> GND_TC
- C8 pad 2: AGND -> GND_TC
- C9 pad 1: AGND -> GND_TC
- D12 pad 2: AGND -> GND_TC
- P4 pad 10: /Fan/TACH_IN -> +3.3V
- P4 pad 11: /Fan/FAN_OUT- -> /PowerAdjustmentMonitor/V-_ADJ
- P4 pad 12: /Fan/FAN_OUT+ -> /PowerAdjustmentMonitor/V+_ADJ
- P4 pad 3: GND -> /Fan/FAN_OUT-
- P4 pad 4: /PowerAdjustmentMonitor/V+_ADJ -> /Fan/FAN_OUT+
- P4 pad 5: /PowerAdjustmentMonitor/V-_ADJ -> /Fan/TACH_IN
- P4 pad 6: +3.3V -> /Thermocouple/TC IN -
- P4 pad 7: +5V -> /Thermocouple/TC IN +
- P4 pad 8: /Thermocouple/TC IN + -> GND
- P4 pad 9: /Thermocouple/TC IN - -> +5V
- Q2 pad S: AGND -> GND_FAN
- Q3 pad 3: GND -> GND_FAN
- R16 pad 2: GND -> GND_FAN
- R17 pad 2: GND -> GND_LED
- R19 pad 2: AGND -> GND_PWR
- R2 pad 2: GND -> GND_RELAY
- R20 pad 2: AGND -> GND_PWR
- R23 pad 1: AGND -> GND_PWR
- R24 pad 2: AGND -> GND_PWR
- R48 pad 1: AGND -> GND_TC
- R49 pad 1: AGND -> GND_TC
- R52 pad 1: AGND -> GND_TC
- R55 pad 1: AGND -> GND_TC
- R6 pad 2: GND -> GND_RELAY
- R7 pad 1: AGND -> GND_TC
- U2 pad 11: AGND -> GND_TC
- U2 pad 8: AGND -> GND_TC
- U3 pad 1: AGND -> GND_TC
- U3 pad 2: AGND -> GND_TC
- U3 pad 5: AGND -> GND_TC
- U5 pad 7: AGND -> GND_FAN
- U7 pad 2: GND -> GND_LED
Routing:
- net GND_FAN: track 0.00 -> 3.05 mm, vias 0 -> 1
- net GND_RELAY: track 0.00 -> 2.55 mm, vias 0 -> 1
- net GND_LED: track 0.00 -> 2.13 mm, vias 0 -> 1
- net GND_TC: track 0.00 -> 1.21 mm, vias 0 -> 1
- added copper zone on GND, net GND_FAN
- added copper zone on GND, net GND_LED
- added copper zone on GND, net GND_PWR
- added copper zone on GND, net GND_RELAY
- added copper zone on GND, net GND_TC

Commit message: Layout Work Session 6
Parts:
- added TP1: CONN_1, Measurement_Points:Measurement_Point_Square-TH_Big, F.Cu at (175.9, 131.4)
- MH (x3): value MountingHole_3mm_RevA_Date21Jun2010 -> (none)
- moved L2 49.5 mm to (159.9, 101.3)
- moved C4 44.8 mm to (164.7, 99.9), turned to 90 degrees
- moved L3 36.6 mm to (159.9, 105.4)
- moved C3 30.0 mm to (164.7, 106.8), turned to 90 degrees
- moved TH3 23.1 mm to (161.8, 152.1), turned to 0 degrees
- moved TH1 19.3 mm to (150.6, 98.6)
- moved U9 11.0 mm to (272.7, 108.1)
- moved MH 10.2 mm to (141.0, 156.6)
- moved MH 10.2 mm to (141.0, 98.4)
- moved D4 9.77 mm to (287.7, 116.8)
- moved U4 7.03 mm to (271.8, 116.7)
- moved Q3 5.99 mm to (290.1, 126.0)
- moved P2 5.59 mm to (257.8, 116.1)
- moved SW1 5.42 mm to (178.3, 98.0)
- moved U8 4.77 mm to (284.6, 108.1)
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Connections:
- C10 pad 1: GND_TC -> AGND
- C11 pad 2: GND_TC -> AGND
- C12 pad 1: GND_FAN -> AGND
- C13 pad 2: GND_FAN -> AGND
- C14 pad 2: GND_TC -> AGND
- C15 pad 1: GND_TC -> AGND
- C20 pad 2: GND_TC -> AGND
- C21 pad 1: GND_TC -> AGND
- C24 pad 2: GND_TC -> AGND
- C25 pad 2: GND_TC -> AGND
- C7 pad 1: GND_TC -> AGND
- C8 pad 2: GND_TC -> AGND
- C9 pad 1: GND_TC -> AGND
- D12 pad 2: GND_TC -> AGND
- P4 pad 8: GND -> GND_PWR
- Q2 pad S: GND_FAN -> AGND
- Q3 pad 3: GND_FAN -> AGND
- R16 pad 2: GND_FAN -> AGND
- R48 pad 1: GND_TC -> AGND
- R49 pad 1: GND_TC -> AGND
- R52 pad 1: GND_TC -> AGND
- R55 pad 1: GND_TC -> AGND
- R7 pad 1: GND_TC -> AGND
- U2 pad 11: GND_TC -> AGND
- U2 pad 8: GND_TC -> AGND
- U3 pad 1: GND_TC -> AGND
- U3 pad 2: GND_TC -> AGND
- U3 pad 5: GND_TC -> AGND
- U5 pad 7: GND_FAN -> AGND
Routing:
- net +12V: track 0.00 -> 210.2 mm, vias 0 -> 1
- net -12V: track 0.00 -> 201.3 mm, vias 0 -> 1
- net +12C: track 0.00 -> 187.6 mm, vias 0 -> 2
- net /Relay/RELAY_COM: track 0.00 -> 22.6 mm
- net /Relay/RELAY_NO: track 0.00 -> 8.84 mm
- net /Relay/RELAY_NC: track 0.00 -> 8.80 mm
- net GND_FAN: track 3.05 -> 0.00 mm, vias 1 -> 0
- net +5V: track 0.00 -> 2.31 mm, vias 0 -> 1
- net +12P: track 0.00 -> 2.29 mm, vias 0 -> 1
- net +5P: track 0.00 -> 2.10 mm, vias 0 -> 1
- net GND_TC: track 1.21 -> 0.00 mm, vias 1 -> 0
- net AGND: track 0.00 -> 1.21 mm, vias 0 -> 1
- added copper zone on PWR, net +12P
- added copper zone on PWR, net +5P
- added copper zone on PWR, net +5V
- added copper zone on GND, net AGND
- removed copper zone on GND, net GND_FAN
- removed copper zone on GND, net GND_TC

Commit message: Layout Work Session 6
Pulled from CE
Parts:
- removed HEATSINK_V8508H (x2): VAL**, BenchBudEE:HEATSINK_V8508H
- removed MH (x3): , Mounting_Holes:MountingHole_3mm
- added 3 mm: VAL**, 3mm-NPTH, F.Cu at (58.9, 79.8)
- added 3 mm: VAL**, 3mm-NPTH, F.Cu at (58.7, 137.4)
- added 3 mm: VAL**, 3mm-NPTH, F.Cu at (207.2, 81.5)
- added JP2: JUMPER, PIN_ARRAY_2X1, F.Cu at (87.6, 108.8)
- added JP3: JUMPER, PIN_ARRAY_2X1, F.Cu at (94.6, 115.5)
- added JP4: JUMPER, PIN_ARRAY_2X1, F.Cu at (87.6, 119.2)
- added V8508H: VAL**, V8508H, F.Cu at (158.0, 79.6)
- added V8508H: VAL**, V8508H, F.Cu at (175.7, 79.3)
- ARD1: footprint BenchBudEE:ARDUINO_SHIELD -> Arduino
- C1, C10, C12, C13, C14, C15, C16, C17, C18, C19, C20, C21, C22, C23, C24, C5, C6, C7, C8: footprint Capacitors_SMD:c_0805 -> SM0805
- C11, C9: footprint Capacitors_SMD:c_0805 -> SM0805; moved to B.Cu
- C2, C3, C4: footprint Capacitors_SMD:c_1206 -> SM1206
- C25: footprint Capacitors_SMD:c_0805 -> SM0805; moved to F.Cu
- D1: footprint LEDs:LED-0603 -> LED-0603
- D10, D11, D12, D3, D6, D7, D8, D9: footprint BenchBudEE:Diode_SOT23 -> SOT23-DIODE; moved to B.Cu
- D2, D4: footprint Diodes_SMD:Diode-SMA_Standard -> SMA
- D5: footprint BenchBudEE:DIODE_SOD-323 -> SOD-323
- JP1: footprint Pin_Headers:Pin_Header_Straight_2x01 -> PIN_ARRAY_2X1
- K1: footprint BenchBudEE:TE-SPDT_RELAY -> TE-SPDT
- L1, L2, L3: footprint SMD_Packages:SM1210L -> SM1210L
- L4: footprint BenchBudEE:INDUCTOR_NR4012T220M -> NR4012
- P1: footprint BenchBudEE:ATX_HEADER -> ATX_Header
- P2: footprint Pin_Headers:Pin_Header_Straight_2x03 -> pin_array_3x2
- P3: footprint Pin_Headers:Pin_Header_Straight_1x02 -> PIN_ARRAY_2X1
- P4: footprint BenchBudEE:12_Pin_3.5mm_TB -> 12pinTB
- P5: footprint BenchBudEE:3_Pin_5mm_TB -> 3pinTB
- Q1: footprint SMD_Packages:SOT23EBC -> SOT23EBC
- Q2: footprint SMD_Packages:SOT23GDS -> SOT23GDS; moved to B.Cu
- Q3, Q4: footprint SMD_Packages:DPAK2 -> DPAK2
- R1, R11, R13, R14, R2, R22, R23, R3, R4, R43, R5, R53, R55, R6: footprint Resistors_SMD:Resistor_SMD0805_HandSoldering -> SM0805
- R10, R16, R7, R8, R9: footprint Resistors_SMD:Resistor_SMD1206_HandSoldering -> SM1206
- R12, R15, R18, R21, R24, R25, R44, R45, R52, R54: footprint Resistors_SMD:Resistor_SMD0805_HandSoldering -> SM0805; moved to F.Cu
- R17, R48, R49: footprint Resistors_SMD:Resistor_SMD0805_HandSoldering -> SM0805; moved to B.Cu
- R19, R20: footprint BenchBudEE:POT-EVUE3K -> EVUE3K
- R26, R27, R28, R29, R30, R31, R32, R33, R34, R35, R36, R37, R38, R39, R40, R41, R42, R46, R47, R50, R51: footprint BenchBudEE:SM0805-Bridge -> SM0805-blob
- SW1: footprint BenchBudEE:SLIDE_SWITCH_SPDT -> BB_switch
- TH1, TH2, TH3, TH4, TH5: footprint SMD_Packages:SM1812 -> SM1812
- TP1: footprint Measurement_Points:Measurement_Point_Square-TH_Big -> 1pin
- U1: footprint BenchBudEE:SMD-4 -> 4-SMD
- U11, U9: value LM317T -> LM317; footprint Power_Integrations:TO-220 -> TO220_VERT
- U2: footprint SMD_Packages:SSOP20 -> SSOP20
- U3: footprint SMD_Packages:SOT353 -> SOT353
- U4: footprint SOIC_Packages:SOIC-14_Narrow -> SO14N
- U5: footprint SMD_Packages:SO8N -> SO8N
- U6, U8: footprint Power_Integrations:TO-220 -> TO220_VERT
- U7: footprint Housings_SOT-23_SOT-143_TSOT-6:TSOT6-MK06A-Housing -> SOT23_6
- moved R24 188.2 mm to (151.3, 94.2), turned to 90 degrees
- moved C23 186.5 mm to (157.0, 89.4), turned to 180 degrees
- moved R23 176.2 mm to (149.2, 94.3)
- moved R15 155.3 mm to (168.2, 112.4)
- moved R49 154.9 mm to (168.8, 98.2), turned to 90 degrees
- moved Q2 152.1 mm to (179.1, 103.6), turned to 270 degrees
- moved R48 151.1 mm to (173.1, 96.3)
- moved JP1 151.0 mm to (94.7, 111.4)
- moved R18 150.5 mm to (140.7, 83.5)
- moved D12 145.7 mm to (202.3, 92.5), turned to 180 degrees
- moved R12 143.7 mm to (186.2, 96.2), turned to 0 degrees
- moved C13 143.0 mm to (184.0, 114.4), turned to 0 degrees
- moved R53 142.6 mm to (202.8, 85.7), turned to 0 degrees
- moved C25 142.2 mm to (200.2, 91.9), turned to 180 degrees
- moved R8 142.1 mm to (188.7, 103.6)
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Connections:
- ARD1 pad 1: Net-(ARD1-Pad1) -> N-0000055
- ARD1 pad 10: Net-(ARD1-Pad10) -> (no net)
- ARD1 pad 11: Net-(ARD1-Pad11) -> N-0000037
- ARD1 pad 12: Net-(ARD1-Pad12) -> N-0000041
- ARD1 pad 13: Net-(ARD1-Pad13) -> N-0000053
- ARD1 pad 2: Net-(ARD1-Pad2) -> N-0000058
- ARD1 pad 3: Net-(ARD1-Pad3) -> N-0000057
- ARD1 pad 4: Net-(ARD1-Pad4) -> N-0000056
- ARD1 pad 5: Net-(ARD1-Pad5) -> N-0000036
- ARD1 pad 6: Net-(ARD1-Pad6) -> N-0000043
- ARD1 pad 7: Net-(ARD1-Pad7) -> N-0000044
- ARD1 pad 8: Net-(ARD1-Pad8) -> N-0000045
- ARD1 pad 9: Net-(ARD1-Pad9) -> (no net)
- C19 pad 1: Net-(C19-Pad1) -> N-00000125
- C20 pad 1: Net-(C20-Pad1) -> N-00000126
- D10 pad 1: Net-(C20-Pad1) -> N-00000126
- D8 pad 1: Net-(C19-Pad1) -> N-00000125
- JP1 pad 1: AGND -> GND
- JP1 pad 2: GND -> AGND
- P1 pad 1: Net-(P1-Pad1) -> (no net)
- P1 pad 11: Net-(P1-Pad11) -> (no net)
- P1 pad 13: Net-(P1-Pad13) -> (no net)
- P1 pad 15: Net-(P1-Pad15) -> (no net)
- P1 pad 17: Net-(P1-Pad17) -> (no net)
- P1 pad 18: Net-(P1-Pad18) -> (no net)
- P1 pad 19: Net-(P1-Pad19) -> (no net)
- P1 pad 20: Net-(P1-Pad20) -> (no net)
- P1 pad 21: Net-(P1-Pad21) -> (no net)
- P1 pad 22: Net-(P1-Pad22) -> (no net)
- P1 pad 23: Net-(P1-Pad23) -> (no net)
- P1 pad 24: Net-(P1-Pad24) -> (no net)
- P1 pad 7: Net-(P1-Pad7) -> (no net)
- P1 pad 8: Net-(P1-Pad8) -> (no net)
- P1 pad 9: Net-(P1-Pad9) -> (no net)
- P4 pad 3: /Fan/FAN_OUT- -> /Fan/TACH_IN
- P4 pad 4: /Fan/FAN_OUT+ -> /Fan/FAN_OUT-
- P4 pad 5: /Fan/TACH_IN -> /Fan/FAN_OUT+
- P4 pad 8: GND_PWR -> +5V
- P4 pad 9: +5V -> GND_PWR
- R20 pad 1: Net-(C19-Pad1) -> N-00000125
- R21 pad 1: Net-(C19-Pad1) -> N-00000125
- R26 pad 1: Net-(ARD1-PadRST) -> N-0000055
- R27 pad 1: Net-(ARD1-PadGND1) -> N-0000058
- R28 pad 1: Net-(ARD1-PadGND2) -> N-0000057
- R29 pad 1: Net-(ARD1-PadV_IN) -> N-0000056
- R30 pad 1: Net-(ARD1-PadAD0) -> N-0000036
- R31 pad 1: Net-(ARD1-PadAD1) -> N-0000043
- R32 pad 1: Net-(ARD1-PadAD2) -> N-0000044
- R33 pad 1: Net-(ARD1-PadAD3) -> N-0000045
- R34 pad 2: Net-(ARD1-Pad13) -> N-0000033
- R35 pad 2: Net-(ARD1-Pad12) -> N-0000032
- R36 pad 2: Net-(ARD1-Pad11) -> N-0000034
- R37 pad 2: Net-(ARD1-Pad10) -> N-0000042
- R38 pad 2: Net-(ARD1-Pad9) -> N-0000040
- R39 pad 2: Net-(ARD1-Pad8) -> N-0000038
- R40 pad 2: Net-(ARD1-Pad7) -> N-0000035
- R41 pad 2: Net-(ARD1-Pad1) -> N-0000041
- R42 pad 2: Net-(ARD1-Pad0) -> N-0000037
- R46 pad 2: Net-(ARD1-Pad5) -> N-0000051
- R47 pad 2: Net-(ARD1-Pad4) -> N-0000046
- R50 pad 2: Net-(ARD1-Pad3) -> N-0000054
- R51 pad 2: Net-(ARD1-Pad2) -> N-0000053
- R54 pad 1: Net-(C20-Pad1) -> N-00000126
- R55 pad 2: Net-(C20-Pad1) -> N-00000126
- U11 pad 1: Net-(C19-Pad1) -> +12V
- U11 pad 2: /PowerAdjustmentMonitor/V+_ADJ -> N-00000125
- U11 pad 3: +12V -> /PowerAdjustmentMonitor/V+_ADJ
- U2 pad 10: REF- -> (no net)
- U2 pad 15: Net-(U2-Pad15) -> (no net)
- U2 pad 16: Net-(U2-Pad16) -> (no net)
- U2 pad 9: REF+ -> (no net)
- U9 pad 1: Net-(C20-Pad1) -> +12V
- U9 pad 2: FE_V+ -> N-00000126
- U9 pad 3: +12V -> FE_V+
Routing:
- net +3.3V: track 0.00 -> 145.5 mm
- net N-00000107: track 0.00 -> 50.3 mm
- net +12P: track 2.29 -> 48.7 mm, vias 1 -> 2
- net GND: track 0.00 -> 32.1 mm
- net -12P: track 0.00 -> 31.6 mm, vias 0 -> 1
- net N-00000102: track 0.00 -> 19.8 mm
- net +5P: track 2.10 -> 10.5 mm, vias 1 -> 2
- net +12V: track 210.2 -> 203.4 mm
- net N-00000103: track 0.00 -> 5.80 mm
- net +5V: track 2.31 -> 7.83 mm, vias 1 -> 2
- net -12V: track 201.3 -> 205.8 mm
- net /Relay/RELAY_COM: track 22.6 -> 24.0 mm
- net /Relay/RELAY_NO: track 8.84 -> 10.2 mm
- net GND_RELAY: track 2.55 -> 1.65 mm
- net /Relay/RELAY_NC: track 8.80 -> 9.62 mm
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- added copper zone on GND, net GND
- removed copper zone on PWR, net +3.3V
Other:
- board text added: "Do we need a second GND?"
