File: Fan.sch (KiCad schematic (older format))
At the start: 9 parts, among them Q2 MOSFET_N, Q3 MOSFET_N, Q4 MOSFET_N, U11 MCP4922-E/SL, U2 OPA4170

Commit message: Associating and Placing the Current/Fan Driver Module
Parts:
- removed U11: MCP4922-E/SL, SO14, symbol MCP4922-E/SL
- added C10, C11: C, symbol C
- added U11: MCP4801, symbol MCP4801
- D5: value DIODE -> B130-13-F; MFG Name (none) -> Diodes Inc; MFG Part Number (none) -> B130-13-F
- Q2: value MOSFET_N -> DMN65D8L-7; MFG Name (none) -> Diodes Inc; MFG Part Number (none) -> DMN65D8L-7
- Q3, Q4: value MOSFET_N -> AOD476; MFG Name (none) -> Alpha & Omega; MFG Part Number (none) -> AOD476
- TH5: value THERMISTOR -> PTC; MFG Name (none) -> TE Connectivity; MFG Part Number (none) -> MINISMDC050F-2
Connections:
- net labels added: +5V, ~LDAC, ~SHDN
- net labels removed: MISO
- wire segments 34 -> 44
Changed lines of the file:
@@
 P 8100 2350
 F 0 "Q4" H 8110 2520 60  0000 R CNN
-F 1 "MOSFET_N" H 8110 2200 60  0000 R CNN
+F 1 "AOD476" H 8110 2200 60  0000 R CNN
 F 2 "" H 8100 2350 60  0000 C CNN
 F 3 "" H 8100 2350 60  0000 C CNN
+F 4 "Alpha & Omega" H 8100 2350 60  0001 C CNN "MFG Name"
+F 5 "AOD476" H 8100 2350 60  0001 C CNN "MFG Part Number"
 	1    8100 2350
 	1    0    0    -1
@@
 	1    0    0    -1
 $EndComp
-Text HLabel 1900 2000 0    60   Output ~ 0
-MISO
-Text HLabel 1900 2200 0    60   Input ~ 0
+Text HLabel 1500 2250 0    60   Input ~ 0
 MOSI
-Text HLabel 1900 2300 0    60   Input ~ 0
+Text HLabel 1500 2150 0    60   Input ~ 0
 SCLK
-Text HLabel 1900 2400 0    60   Input ~ 0
+Text HLabel 1500 2050 0    60   Input ~ 0
 ~CS
 Text HLabel 1750 3700 0    60   Output ~ 0
@@
 $EndComp
 $Comp
-L MCP4922-E/SL U11
-U 1 1 52F15F05
-P 2750 2400
-F 0 "U11" H 2900 2800 40  0000 L BNN
-F 1 "MCP4922-E/SL" H 2900 2750 40  0000 L BNN
-F 2 "SO14" H 2750 2400 30  0000 C CIN
-F 3 "" H 2750 2400 60  0000 C CNN
-	1    2750 2400
-	1    0    0    -1
-$EndComp
-$Comp
 L THERMISTOR TH5
 U 1 1 52F82F82
 P 8200 1150
 F 0 "TH5" V 8300 1200 50  0000 C CNN
-F 1 "THERMISTOR" V 8100 1150 50  0000 C CNN
+F 1 "PTC" V 8100 1150 50  0000 C CNN
 F 2 "" H 8200 1150 60  0000 C CNN
 F 3 "" H 8200 1150 60  0000 C CNN
+F 4 "TE Connectivity" H 8200 1150 60  0001 C CNN "MFG Name"
+F 5 "MINISMDC050F-2" H 8200 1150 60  0001 C CNN "MFG Part Number"
 	1    8200 1150
 	1    0    0    -1
@@
 P 7800 1750
 F 0 "D5" H 7800 1850 40  0000 C CNN
-F 1 "DIODE" H 7800 1650 40  0000 C CNN
+F 1 "B130-13-F" H 7800 1650 40  0000 C CNN
 F 2 "" H 7800 1750 60  0000 C CNN
 F 3 "" H 7800 1750 60  0000 C CNN
+F 4 "Diodes Inc" H 7800 1750 60  0001 C CNN "MFG Name"
+F 5 "B130-13-F" H 7800 1750 60  0001 C CNN "MFG Part Number"
 	1    7800 1750
 	0    -1   -1   0
@@
 P 7750 4250
 F 0 "Q3" H 7760 4420 60  0000 R CNN
-F 1 "MOSFET_N" H 7760 4100 60  0000 R CNN
+F 1 "AOD476" H 7760 4100 60  0000 R CNN
 F 2 "" H 7750 4250 60  0000 C CNN
 F 3 "" H 7750 4250 60  0000 C CNN
+F 4 "Alpha & Omega" H 7750 4250 60  0001 C CNN "MFG Name"
+F 5 "AOD476" H 7750 4250 60  0001 C CNN "MFG Part Number"
 	1    7750 4250
 	1    0    0    -1
@@
 Connection ~ 8200 3700
 Wire Wire Line
-	1900 2200 2200 2200
-Wire Wire Line
-	1900 2300 2200 2300
-Wire Wire Line
-	1900 2400 2200 2400
+	1500 2250 1800 2250
+Wire Wire Line
+	1500 2150 1800 2150
+Wire Wire Line
+	1500 2050 1800 2050
 Wire Wire Line
 	3300 2250 3800 2250
@@
 P 4700 2600
 F 0 "Q2" H 4710 2770 60  0000 R CNN
-F 1 "MOSFET_N" H 4710 2450 60  0000 R CNN
+F 1 "DMN65D8L-7" H 4710 2450 60  0000 R CNN
 F 2 "" H 4700 2600 60  0000 C CNN
 F 3 "" H 4700 2600 60  0000 C CNN
+F 4 "Diodes Inc" H 4700 2600 60  0001 C CNN "MFG Name"
+F 5 "DMN65D8L-7" H 4700 2600 60  0001 C CNN "MFG Part Number"
 	1    4700 2600
 	1    0    0    -1
@@
 	1    0    0    -1
 $EndComp
+$Comp
+L MCP4801 U11
+U 1 1 530AA580
+P 2500 2250
+F 0 "U11" H 2650 1900 60  0000 C CNN
+F 1 "MCP4801" H 2550 2250 60  0000 C CNN
+F 2 "" H 2500 2250 60  0000 C CNN
+F 3 "" H 2500 2250 60  0000 C CNN
+	1    2500 2250
+	1    0    0    -1
+$EndComp
+Text HLabel 1500 2350 0    60   Input ~ 0
+~LDAC
+Text HLabel 1500 2450 0    60   Input ~ 0
+~SHDN
+Wire Wire Line
+	1500 2350 1800 2350
+Wire Wire Line
+	1500 2450 1800 2450
+$Comp
+L C C10
+U 1 1 530B47E4
+P 2150 1550
+F 0 "C10" H 2150 1650 40  0000 L CNN
+F 1 "C" H 2156 1465 40  0000 L CNN
+F 2 "" H 2188 1400 30  0000 C CNN
+F 3 "" H 2150 1550 60  0000 C CNN
+	1    2150 1550
+	0    1    -1   0
+$EndComp
+$Comp
+L AGND #PWR064
+U 1 1 530B47EA
+P 1850 1800
+F 0 "#PWR064" H 1850 1800 40  0001 C CNN
+F 1 "AGND" H 1850 1730 50  0000 C CNN
+F 2 "" H 1850 1800 60  0000 C CNN
+F 3 "" H 1850 1800 60  0000 C CNN
+	1    1850 1800
+	-1   0    0    -1
+$EndComp
+Wire Wire Line
+	2350 1550 2500 1550
+Wire Wire Line
+	2500 1400 2500 1650
+$Comp
+L +5V #PWR065
+U 1 1 530B47F5
+P 2500 1400
+F 0 "#PWR065" H 2500 1490 20  0001 C CNN
+F 1 "+5V" H 2500 1490 30  0000 C CNN
+F 2 "" H 2500 1400 60  0000 C CNN
+F 3 "" H 2500 1400 60  0000 C CNN
+	1    2500 1400
+	1    0    0    -1
+$EndComp
+Connection ~ 2500 1550
+$Comp
+L AGND #PWR066
+U 1 1 530B47FC
+P 2500 3050
+F 0 "#PWR066" H 2500 3050 40  0001 C CNN
+F 1 "AGND" H 2500 2980 50  0000 C CNN
+F 2 "" H 2500 3050 60  0000 C CNN
+F 3 "" H 2500 3050 60  0000 C CNN
+	1    2500 3050
+	1    0    0    -1
+$EndComp
+Wire Wire Line
+	2500 3050 2500 2850
+Wire Wire Line
+	8450 850  8200 850
+Connection ~ 8200 850
+Wire Wire Line
+	1950 1550 1850 1550
+Wire Wire Line
+	1850 1550 1850 1800
+$Comp
+L C C11
+U 1 1 530B51B3
+P 8650 850
+F 0 "C11" H 8650 950 40  0000 L CNN
+F 1 "C" H 8656 765 40  0000 L CNN
+F 2 "" H 8688 700 30  0000 C CNN
+F 3 "" H 8650 850 60  0000 C CNN
+	1    8650 850
+	0    -1   -1   0
+$EndComp
+$Comp
+L AGND #PWR067
+U 1 1 530B51C8
+P 9000 1050
+F 0 "#PWR067" H 9000 1050 40  0001 C CNN
+F 1 "AGND" H 9000 980 50  0000 C CNN
+F 2 "" H 9000 1050 60  0000 C CNN
+F 3 "" H 9000 1050 60  0000 C CNN
+	1    9000 1050
+	1    0    0    -1
+$EndComp
+Wire Wire Line
+	8850 850  9000 850
+Wire Wire Line
+	9000 850  9000 1050
 $EndSCHEMATC

Commit message: Merge CE BenchBudEE commit 00937c39d96b9ebb1b0292c11cc231788ab24edd
Parts:
- removed C10, C11: C, symbol C
- removed D5: B130-13-F, symbol DIODE
- removed Q3, Q4: AOD476, symbol MOSFET_N
- removed R41, R42: R, symbol R
- removed U11: MCP4801, symbol MCP4801
- removed U2: OPA4170, symbol LM324
- added C12, C13: C, ~, symbol C
- added D4: B130-13-F, ~, symbol DIODE
- added Q3, Q4: AOD476, ~, symbol MOS_N_NUM
- added R15, R16: R, ~, symbol R
- added U4: OPA4170, symbol LM324
- added U5: MCP4801, symbol MCP4801
- Q2: footprint (none) -> ~
- TH5: value PTC -> MINISMDC050F-2; footprint (none) -> ~
Connections:
- net labels added: CS_N, FE_V+, FE_V-, GND
- net labels removed: +12V, -12V, ~CS
- wire segments 44 -> 45

Commit message: Layout Work Session 4
Connections:
- net labels added: GND_FAN
- net labels removed: AGND, GND
Changed lines of the file:
@@
-	1    0    0    -1
-$EndComp
-$Comp
-L AGND #PWR033
-U 1 1 523698EE
-P 4700 3750
-F 0 "#PWR033" H 4700 3750 40  0001 C CNN
-F 1 "AGND" H 4700 3680 50  0000 C CNN
-F 2 "" H 4700 3750 60  0000 C CNN
-F 3 "" H 4700 3750 60  0000 C CNN
-	1    4700 3750
 	1    0    0    -1
 $EndComp
@@
 FAN_MODE
 $Comp
-L +12C #PWR034
+L +12C #PWR030
 U 1 1 5243907A
 P 7900 1000
-F 0 "#PWR034" H 7900 970 30  0001 C CNN
+F 0 "#PWR030" H 7900 970 30  0001 C CNN
 F 1 "+12C" H 7900 1110 40  0000 C CNN
 F 2 "~" H 7900 1000 60  0000 C CNN
@@
 	2000 1950 1900 1950
 Connection ~ 2000 1950
-$Comp
-L AGND #PWR035
-U 1 1 525C14F8
-P 1350 2050
-F 0 "#PWR035" H 1350 2050 40  0001 C CNN
-F 1 "AGND" H 1350 1980 50  0000 C CNN
-F 2 "" H 1350 2050 60  0000 C CNN
-F 3 "" H 1350 2050 60  0000 C CNN
-	1    1350 2050
-	1    0    0    -1
-$EndComp
 Wire Wire Line
 	1350 2050 1350 1950
@@
 	1350 1950 1500 1950
 $Comp
-L +5V #PWR036
+L +5V #PWR031
 U 1 1 525C1500
 P 2000 1700
-F 0 "#PWR036" H 2000 1790 20  0001 C CNN
+F 0 "#PWR031" H 2000 1790 20  0001 C CNN
 F 1 "+5V" H 2000 1790 30  0000 C CNN
 F 2 "~" H 2000 1700 60  0000 C CNN
 F 3 "~" H 2000 1700 60  0000 C CNN
 	1    2000 1700
-	1    0    0    -1
-$EndComp
-$Comp
-L AGND #PWR037
-U 1 1 525C1506
-P 2000 3950
-F 0 "#PWR037" H 2000 3950 40  0001 C CNN
-F 1 "AGND" H 2000 3880 50  0000 C CNN
-F 2 "" H 2000 3950 60  0000 C CNN
-F 3 "" H 2000 3950 60  0000 C CNN
-	1    2000 3950
 	1    0    0    -1
 $EndComp
@@
 $EndComp
 $Comp
-L FE_V+ #PWR038
+L FE_V+ #PWR032
 U 1 1 526E03BB
 P 6150 2550
-F 0 "#PWR038" H 6150 2650 30  0001 C CNN
+F 0 "#PWR032" H 6150 2650 30  0001 C CNN
 F 1 "FE_V+" H 6150 2650 30  0000 C CNN
 F 2 "~" H 6150 2550 60  0000 C CNN
@@
 	6150 2700 6150 2550
 $Comp
-L GND #PWR039
-U 1 1 526E2673
+L GND_FAN #PWR033
+U 1 1 5313DCC7
+P 8600 1400
+F 0 "#PWR033" H 8600 1400 30  0001 C CNN
+F 1 "GND_FAN" H 8600 1330 30  0000 C CNN
+F 2 "" H 8600 1400 60  0000 C CNN
+F 3 "" H 8600 1400 60  0000 C CNN
+	1    8600 1400
+	1    0    0    -1
+$EndComp
+$Comp
+L GND_FAN #PWR034
+U 1 1 5313DCE5
 P 7900 5550
-F 0 "#PWR039" H 7900 5550 30  0001 C CNN
-F 1 "GND" H 7900 5480 30  0001 C CNN
-F 2 "~" H 7900 5550 60  0000 C CNN
-F 3 "~" H 7900 5550 60  0000 C CNN
+F 0 "#PWR034" H 7900 5550 30  0001 C CNN
+F 1 "GND_FAN" H 7900 5480 30  0000 C CNN
+F 2 "" H 7900 5550 60  0000 C CNN
+F 3 "" H 7900 5550 60  0000 C CNN
 	1    7900 5550
 	1    0    0    -1
 $EndComp
 $Comp
-L GND #PWR040
-U 1 1 526E268A
-P 8600 1400
-F 0 "#PWR040" H 8600 1400 30  0001 C CNN
-F 1 "GND" H 8600 1330 30  0001 C CNN
-F 2 "~" H 8600 1400 60  0000 C CNN
-F 3 "~" H 8600 1400 60  0000 C CNN
-	1    8600 1400
-	1    0    0    -1
-$EndComp
+L GND_FAN #PWR035
+U 1 1 5313DCF9
+P 4700 3750
+F 0 "#PWR035" H 4700 3750 30  0001 C CNN
+F 1 "GND_FAN" H 4700 3680 30  0000 C CNN
+F 2 "" H 4700 3750 60  0000 C CNN
+F 3 "" H 4700 3750 60  0000 C CNN
+	1    4700 3750
+	1    0    0    -1
+$EndComp
+$Comp
+L GND_FAN #PWR036
+U 1 1 5313DD0D
+P 2000 3950
+F 0 "#PWR036" H 2000 3950 30  0001 C CNN
+F 1 "GND_FAN" H 2000 3880 30  0000 C CNN
+F 2 "" H 2000 3950 60  0000 C CNN
+F 3 "" H 2000 3950 60  0000 C CNN
+	1    2000 3950
+	1    0    0    -1
+$EndComp
+$Comp
+L GND_FAN #PWR037
+U 1 1 5313DD21
+P 1350 2050
+F 0 "#PWR037" H 1350 2050 30  0001 C CNN
+F 1 "GND_FAN" H 1350 1980 30  0000 C CNN
+F 2 "" H 1350 2050 60  0000 C CNN
+F 3 "" H 1350 2050 60  0000 C CNN
+	1    1350 2050
+	1    0    0    -1
+$EndComp

Commit message: Layout Work Session 6
Connections:
- net labels added: AGND
- net labels removed: GND_FAN
Changed lines of the file:
@@
 	6150 2700 6150 2550
 $Comp
-L GND_FAN #PWR033
-U 1 1 5313DCC7
+L AGND #PWR033
+U 1 1 53147078
 P 8600 1400
-F 0 "#PWR033" H 8600 1400 30  0001 C CNN
-F 1 "GND_FAN" H 8600 1330 30  0000 C CNN
+F 0 "#PWR033" H 8600 1400 40  0001 C CNN
+F 1 "AGND" H 8600 1330 50  0000 C CNN
 F 2 "" H 8600 1400 60  0000 C CNN
 F 3 "" H 8600 1400 60  0000 C CNN
@@
 $EndComp
 $Comp
-L GND_FAN #PWR034
-U 1 1 5313DCE5
+L AGND #PWR034
+U 1 1 53147096
 P 7900 5550
-F 0 "#PWR034" H 7900 5550 30  0001 C CNN
-F 1 "GND_FAN" H 7900 5480 30  0000 C CNN
+F 0 "#PWR034" H 7900 5550 40  0001 C CNN
+F 1 "AGND" H 7900 5480 50  0000 C CNN
 F 2 "" H 7900 5550 60  0000 C CNN
 F 3 "" H 7900 5550 60  0000 C CNN
@@
 $EndComp
 $Comp
-L GND_FAN #PWR035
-U 1 1 5313DCF9
+L AGND #PWR035
+U 1 1 531470AA
 P 4700 3750
-F 0 "#PWR035" H 4700 3750 30  0001 C CNN
-F 1 "GND_FAN" H 4700 3680 30  0000 C CNN
+F 0 "#PWR035" H 4700 3750 40  0001 C CNN
+F 1 "AGND" H 4700 3680 50  0000 C CNN
 F 2 "" H 4700 3750 60  0000 C CNN
 F 3 "" H 4700 3750 60  0000 C CNN
@@
 $EndComp
 $Comp
-L GND_FAN #PWR036
-U 1 1 5313DD0D
+L AGND #PWR036
+U 1 1 531470BE
 P 2000 3950
-F 0 "#PWR036" H 2000 3950 30  0001 C CNN
-F 1 "GND_FAN" H 2000 3880 30  0000 C CNN
+F 0 "#PWR036" H 2000 3950 40  0001 C CNN
+F 1 "AGND" H 2000 3880 50  0000 C CNN
 F 2 "" H 2000 3950 60  0000 C CNN
 F 3 "" H 2000 3950 60  0000 C CNN
@@
 $EndComp
 $Comp
-L GND_FAN #PWR037
-U 1 1 5313DD21
+L AGND #PWR037
+U 1 1 531470D2
 P 1350 2050
-F 0 "#PWR037" H 1350 2050 30  0001 C CNN
-F 1 "GND_FAN" H 1350 1980 30  0000 C CNN
+F 0 "#PWR037" H 1350 2050 40  0001 C CNN
+F 1 "AGND" H 1350 1980 50  0000 C CNN
 F 2 "" H 1350 2050 60  0000 C CNN
 F 3 "" H 1350 2050 60  0000 C CNN
