File: LED_Driver.sch (KiCad schematic (older format))
At the start: 6 parts, among them U10 AP5726

Commit message: Merge CE BenchBudEE commit 00937c39d96b9ebb1b0292c11cc231788ab24edd
Parts:
- removed C4: C, symbol C
- removed D4: DIODESCH, symbol DIODESCH
- removed L3: INDUCTOR, symbol INDUCTOR
- removed R40: R, symbol R
- removed U10: AP5726, symbol AP5726
- added C6: 1U, ~, symbol C
- added D5: B0540WS-7, ~, symbol DIODESCH
- added L4: 22u, ~, symbol INDUCTOR
- added R17: 15, ~, symbol R
- added U7: AP5726, symbol AP5726
- C5: value C -> 1U; footprint (none) -> ~
Connections:
- net labels added: +5P
- net labels removed: +5V
- wire segments 19 -> 22

Commit message: Layout Work Session 4
Connections:
- net GND renamed GND_LED
Changed lines of the file:
@@
 Wire Wire Line
 	2150 2950 2850 2950
-$Comp
-L GND #PWR016
-U 1 1 523F5D68
-P 2550 2350
-F 0 "#PWR016" H 2550 2350 30  0001 C CNN
-F 1 "GND" H 2550 2280 30  0001 C CNN
-F 2 "~" H 2550 2350 60  0000 C CNN
-F 3 "~" H 2550 2350 60  0000 C CNN
-	1    2550 2350
-	1    0    0    -1
-$EndComp
-$Comp
-L GND #PWR017
-U 1 1 523F5D75
-P 3650 4150
-F 0 "#PWR017" H 3650 4150 30  0001 C CNN
-F 1 "GND" H 3650 4080 30  0001 C CNN
-F 2 "~" H 3650 4150 60  0000 C CNN
-F 3 "~" H 3650 4150 60  0000 C CNN
-	1    3650 4150
-	1    0    0    -1
-$EndComp
 Wire Wire Line
 	3650 4150 3650 3900
@@
 Wire Wire Line
 	9400 1650 9400 1900
-$Comp
-L GND #PWR018
-U 1 1 523F5E22
-P 9400 2450
-F 0 "#PWR018" H 9400 2450 30  0001 C CNN
-F 1 "GND" H 9400 2380 30  0001 C CNN
-F 2 "~" H 9400 2450 60  0000 C CNN
-F 3 "~" H 9400 2450 60  0000 C CNN
-	1    9400 2450
-	1    0    0    -1
-$EndComp
 Wire Wire Line
 	9400 2300 9400 2450
@@
 	1    0    0    -1
 $EndComp
+$Comp
+L GND_LED #PWR016
+U 1 1 5313E39D
+P 9400 2450
+F 0 "#PWR016" H 9400 2450 30  0001 C CNN
+F 1 "GND_LED" H 9400 2380 30  0000 C CNN
+F 2 "" H 9400 2450 60  0000 C CNN
+F 3 "" H 9400 2450 60  0000 C CNN
+	1    9400 2450
+	1    0    0    -1
+$EndComp
+$Comp
+L GND_LED #PWR017
+U 1 1 5313E3B1
+P 2550 2350
+F 0 "#PWR017" H 2550 2350 30  0001 C CNN
+F 1 "GND_LED" H 2550 2280 30  0000 C CNN
+F 2 "" H 2550 2350 60  0000 C CNN
+F 3 "" H 2550 2350 60  0000 C CNN
+	1    2550 2350
+	1    0    0    -1
+$EndComp
+$Comp
+L GND_LED #PWR018
+U 1 1 5313E3C5
+P 3650 4150
+F 0 "#PWR018" H 3650 4150 30  0001 C CNN
+F 1 "GND_LED" H 3650 4080 30  0000 C CNN
+F 2 "" H 3650 4150 60  0000 C CNN
+F 3 "" H 3650 4150 60  0000 C CNN
+	1    3650 4150
+	1    0    0    -1
+$EndComp
