File: PowerAdjustmentMonitor.sch (KiCad schematic (older format))
At the start: 37 parts, among them U11 LM317, U6 LM337T, U8 LM337T, U9 LM317

Commit message: Layout Work Session 2
Parts:
- removed U11, U9: LM317, ~, symbol LM317
- added U11, U9: LM317T, TO-220, symbol LM317T
Changed lines of the file:
@@
 LIBS:valves
 LIBS:BenchBuddy
+LIBS:arduino_shieldsNCL
 LIBS:BenchBuddy-cache
 EELAYER 24 0
@@
 $EndDescr
 $Comp
-L +3.3V #PWR37
+L +3.3V #PWR021
 U 1 1 523E00C5
 P 9000 2250
-F 0 "#PWR37" H 9000 2210 30  0001 C CNN
+F 0 "#PWR021" H 9000 2210 30  0001 C CNN
 F 1 "+3.3V" H 9000 2360 30  0000 C CNN
 F 2 "" H 9000 2250 60  0000 C CNN
@@
 $EndComp
 $Comp
-L +5V #PWR36
+L +5V #PWR022
 U 1 1 523E00CB
 P 8700 2250
-F 0 "#PWR36" H 8700 2340 20  0001 C CNN
+F 0 "#PWR022" H 8700 2340 20  0001 C CNN
 F 1 "+5V" H 8700 2340 30  0000 C CNN
 F 2 "" H 8700 2250 60  0000 C CNN
@@
 $EndComp
 $Comp
-L -12V #PWR27
+L -12V #PWR023
 U 1 1 523E0153
 P 1750 5300
-F 0 "#PWR27" H 1750 5430 20  0001 C CNN
+F 0 "#PWR023" H 1750 5430 20  0001 C CNN
 F 1 "-12V" H 1750 5400 30  0000 C CNN
 F 2 "" H 1750 5300 60  0000 C CNN
@@
 $EndComp
 $Comp
-L +12V #PWR29
+L +12V #PWR024
 U 1 1 523E015D
 P 2200 700
-F 0 "#PWR29" H 2200 650 20  0001 C CNN
+F 0 "#PWR024" H 2200 650 20  0001 C CNN
 F 1 "+12V" H 2200 800 30  0000 C CNN
 F 2 "" H 2200 700 60  0000 C CNN
@@
 $EndComp
 $Comp
-L GND #PWR25
+L GND #PWR025
 U 1 1 523E06F9
 P 750 4250
-F 0 "#PWR25" H 750 4250 30  0001 C CNN
+F 0 "#PWR025" H 750 4250 30  0001 C CNN
 F 1 "GND" H 750 4180 30  0001 C CNN
 F 2 "~" H 750 4250 60  0000 C CNN
@@
 $EndComp
 $Comp
-L AGND #PWR26
+L AGND #PWR026
 U 1 1 523E08B2
 P 1350 4250
-F 0 "#PWR26" H 1350 4250 40  0001 C CNN
+F 0 "#PWR026" H 1350 4250 40  0001 C CNN
 F 1 "AGND" H 1350 4180 50  0000 C CNN
 F 2 "~" H 1350 4250 60  0000 C CNN
@@
 $EndComp
 $Comp
-L AGND #PWR28
+L AGND #PWR027
 U 1 1 52562CAD
 P 1900 4250
-F 0 "#PWR28" H 1900 4250 40  0001 C CNN
+F 0 "#PWR027" H 1900 4250 40  0001 C CNN
 F 1 "AGND" H 1900 4180 50  0000 C CNN
 F 2 "~" H 1900 4250 60  0000 C CNN
@@
 $EndComp
 $Comp
-L FE_V+ #PWR34
+L FE_V+ #PWR028
 U 1 1 523E0975
 P 5600 2700
-F 0 "#PWR34" H 5600 2800 30  0001 C CNN
+F 0 "#PWR028" H 5600 2800 30  0001 C CNN
 F 1 "FE_V+" H 5600 2800 30  0000 C CNN
 F 2 "~" H 5600 2700 60  0000 C CNN
@@
 $EndComp
 $Comp
-L LM317 U11
-U 1 1 523E0B74
-P 3350 1000
-F 0 "U11" H 3350 1300 60  0000 C CNN
-F 1 "LM317" H 3400 750 60  0000 L CNN
-F 2 "~" H 3350 1000 60  0000 C CNN
-F 3 "~" H 3350 1000 60  0000 C CNN
-	1    3350 1000
-	1    0    0    -1
-$EndComp
-$Comp
 L R R21
 U 1 1 523E0B81
@@
 $EndComp
 $Comp
-L AGND #PWR33
+L AGND #PWR029
 U 1 1 523E0B8A
 P 3950 2150
-F 0 "#PWR33" H 3950 2150 40  0001 C CNN
+F 0 "#PWR029" H 3950 2150 40  0001 C CNN
 F 1 "AGND" H 3950 2080 50  0000 C CNN
 F 2 "~" H 3950 2150 60  0000 C CNN
@@
 $EndComp
 $Comp
-L LM317 U9
-U 1 1 525F3FCD
-P 3800 3000
-F 0 "U9" H 3800 3300 60  0000 C CNN
-F 1 "LM317" H 3850 2750 60  0000 L CNN
-F 2 "~" H 3800 3000 60  0000 C CNN
-F 3 "~" H 3800 3000 60  0000 C CNN
-	1    3800 3000
-	1    0    0    -1
-$EndComp
-$Comp
 L R R55
 U 1 1 525F3FD3
@@
 $EndComp
 $Comp
-L AGND #PWR32
+L AGND #PWR030
 U 1 1 525F46F5
 P 3800 6100
-F 0 "#PWR32" H 3800 6100 40  0001 C CNN
+F 0 "#PWR030" H 3800 6100 40  0001 C CNN
 F 1 "AGND" H 3800 6030 50  0000 C CNN
 F 2 "~" H 3800 6100 60  0000 C CNN
@@
 $EndComp
 $Comp
-L AGND #PWR31
+L AGND #PWR031
 U 1 1 525F5284
 P 2900 1600
-F 0 "#PWR31" H 2900 1600 40  0001 C CNN
+F 0 "#PWR031" H 2900 1600 40  0001 C CNN
 F 1 "AGND" H 2900 1530 50  0000 C CNN
 F 2 "~" H 2900 1600 60  0000 C CNN
@@
 $EndComp
 $Comp
-L AGND #PWR30
+L AGND #PWR032
 U 1 1 525F532F
 P 2600 6450
-F 0 "#PWR30" H 2600 6450 40  0001 C CNN
+F 0 "#PWR032" H 2600 6450 40  0001 C CNN
 F 1 "AGND" H 2600 6380 50  0000 C CNN
 F 2 "~" H 2600 6450 60  0000 C CNN
@@
 	3950 2000 3950 2150
 Wire Wire Line
-	3350 1350 3350 1450
+	3350 1150 3350 1450
 Wire Wire Line
 	3350 1450 4300 1450
@@
 	2200 2850 3400 2850
 Wire Wire Line
-	3800 3350 3800 3450
+	3800 3150 3800 3450
 Wire Wire Line
 	5600 2850 5600 2700
@@
 Connection ~ 5350 4050
 Wire Wire Line
-	5200 6300 5200 5600
+	5200 5600 5200 6300
 Connection ~ 5200 5600
 Wire Wire Line
@@
 $EndComp
 Connection ~ 4400 4050
+$Comp
+L LM317T U11
+U 1 1 530F1CBE
+P 3350 900
+F 0 "U11" H 3150 1100 40  0000 C CNN
+F 1 "LM317T" H 3350 1100 40  0000 L CNN
+F 2 "TO-220" H 3350 1000 30  0000 C CIN
+F 3 "" H 3350 900 60  0000 C CNN
+	1    3350 900
+	1    0    0    -1
+$EndComp
+$Comp
+L LM317T U9
+U 1 1 530F1D30
+P 3800 2900
+F 0 "U9" H 3600 3100 40  0000 C CNN
+F 1 "LM317T" H 3800 3100 40  0000 L CNN
+F 2 "TO-220" H 3800 3000 30  0000 C CIN
+F 3 "" H 3800 2900 60  0000 C CNN
+	1    3800 2900
+	1    0    0    -1
+$EndComp
 $EndSCHEMATC

Commit message: Layout Work Session 4
Parts:
- removed JP1: JUMPER, ~, symbol JUMPER
Connections:
- net labels added: GND_PWR, GND_TC
- net labels removed: AGND, GND
- wire segments 105 -> 96
Other:
- moved on the sheet: C14, C15, C16, C17, C18, C19, C20, C21, C22, C23, C24, C25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

Commit message: Layout Work Session 6
Connections:
- net labels added: AGND
- net labels removed: GND_TC
Changed lines of the file:
@@
 $EndComp
 $Comp
-L GND_TC #PWR028
-U 1 1 53144567
-P 900 3000
-F 0 "#PWR028" H 900 3000 30  0001 C CNN
-F 1 "GND_TC" H 900 2930 30  0000 C CNN
-F 2 "" H 900 3000 60  0000 C CNN
-F 3 "" H 900 3000 60  0000 C CNN
-	1    900  3000
-	1    0    0    -1
-$EndComp
-$Comp
-L GND_PWR #PWR029
+L GND_PWR #PWR028
 U 1 1 53145CF5
 P 6450 3225
-F 0 "#PWR029" H 6450 3225 30  0001 C CNN
+F 0 "#PWR028" H 6450 3225 30  0001 C CNN
 F 1 "GND_PWR" H 6450 3155 30  0000 C CNN
 F 2 "" H 6450 3225 60  0000 C CNN
@@
 Connection ~ 9575 4375
 Connection ~ 9575 2875
+$Comp
+L AGND #PWR029
+U 1 1 5314869E
+P 900 3000
+F 0 "#PWR029" H 900 3000 40  0001 C CNN
+F 1 "AGND" H 900 2930 50  0000 C CNN
+F 2 "" H 900 3000 60  0000 C CNN
+F 3 "" H 900 3000 60  0000 C CNN
+	1    900  3000
+	1    0    0    -1
+$EndComp
 $EndSCHEMATC

Commit message: Layout Work Session 6
Pulled from CE
Parts:
- removed U11, U9: LM317T, TO-220, symbol LM317T
- added U11, U9: LM317, ~, symbol LM317
Connections:
- wire segments 96 -> 103
Other:
- moved on the sheet: C14, C15, C16, C17, C18, C19, C20, C21, C22, C23, C24, C25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
