File: Thermocouple.sch (KiCad schematic (older format))
At the start: 21 parts, among them P2 CONN_3X2, P3 CONN_2, U1 MCP3901, U2 OPA4170, U3 LMT84

Commit message: Merge CE BenchBudEE commit 00937c39d96b9ebb1b0292c11cc231788ab24edd
Parts:
- removed C6: C, symbol C
- removed R16, R17, R18, R19, R20, R21, R22, R43: R, symbol R
- removed R47: 0, symbol R
- removed U1: MCP3901, symbol MCP3901
- removed U2: OPA4170, symbol LM324
- added C10, C11: C, ~, symbol C
- added R10, R11, R12, R13, R45, R7, R8, R9: R, ~, symbol R
- added R49: 0, ~, symbol R
- added U2: MCP3901, symbol MCP3901
- added U4: OPA4170, symbol LM324
- C1, C7, C8, C9, R44, R48: footprint (none) -> ~
Connections:
- net labels added: FE_V+, FE_V-, TC IN +, TC IN -
- net labels removed: +12V, -12V, TC_IN+, TC_IN-
- wire segments 94 -> 91
Other:
- note added: "16-24Bit ADC"
- note added: "Instrumentation Amp"
- note added: "TEMP SENSOR"
- note removed: "16-24 Bit ADC"
- note removed: "Instrumentation Amplifier"
- note removed: "Temperature Sensor"

Commit message: Layout Work Session 4
Connections:
- net AGND renamed GND_TC
Changed lines of the file:
@@
 Wire Wire Line
 	9000 5000 9000 4850
-$Comp
-L AGND #PWR01
-U 1 1 52364808
-P 4900 4700
-F 0 "#PWR01" H 4900 4700 40  0001 C CNN
-F 1 "AGND" H 4900 4630 50  0000 C CNN
-F 2 "" H 4900 4700 60  0000 C CNN
-F 3 "" H 4900 4700 60  0000 C CNN
-	1    4900 4700
-	1    0    0    -1
-$EndComp
 Wire Wire Line
 	4900 4450 5100 4450
@@
 	5700 6800 5700 6650
 Connection ~ 5600 6800
-$Comp
-L AGND #PWR02
-U 1 1 525797B7
-P 4800 6900
-F 0 "#PWR02" H 4800 6900 40  0001 C CNN
-F 1 "AGND" H 4800 6830 50  0000 C CNN
-F 2 "" H 4800 6900 60  0000 C CNN
-F 3 "" H 4800 6900 60  0000 C CNN
-	1    4800 6900
-	1    0    0    -1
-$EndComp
-Wire Wire Line
-	4800 6900 4800 6800
 Connection ~ 4800 6800
 $Comp
-L +5V #PWR03
+L +5V #PWR01
 U 1 1 5257A1D1
 P 5600 5000
-F 0 "#PWR03" H 5600 5090 20  0001 C CNN
+F 0 "#PWR01" H 5600 5090 20  0001 C CNN
 F 1 "+5V" H 5600 5090 30  0000 C CNN
 F 2 "~" H 5600 5000 60  0000 C CNN
@@
 Connection ~ 6250 3800
 $Comp
-L AGND #PWR04
-U 1 1 5257A2EE
-P 5550 4000
-F 0 "#PWR04" H 5550 4000 40  0001 C CNN
-F 1 "AGND" H 5550 3930 50  0000 C CNN
-F 2 "" H 5550 4000 60  0000 C CNN
-F 3 "" H 5550 4000 60  0000 C CNN
-	1    5550 4000
-	1    0    0    -1
-$EndComp
-$Comp
 L C C10
 U 1 1 5257A357
@@
 	0    -1   -1   0
 $EndComp
-$Comp
-L AGND #PWR05
-U 1 1 5257A35E
-P 5600 2800
-F 0 "#PWR05" H 5600 2800 40  0001 C CNN
-F 1 "AGND" H 5600 2730 50  0000 C CNN
-F 2 "" H 5600 2800 60  0000 C CNN
-F 3 "" H 5600 2800 60  0000 C CNN
-	1    5600 2800
-	1    0    0    -1
-$EndComp
 Wire Wire Line
 	6100 2650 6250 2650
@@
 	6050 3800 6250 3800
 $Comp
-L +5V #PWR06
+L +5V #PWR02
 U 1 1 5257A5A4
 P 5600 5000
-F 0 "#PWR06" H 5600 5090 20  0001 C CNN
+F 0 "#PWR02" H 5600 5090 20  0001 C CNN
 F 1 "+5V" H 5600 5090 30  0000 C CNN
 F 2 "~" H 5600 5000 60  0000 C CNN
@@
 $EndComp
 $Comp
-L +5V #PWR07
+L +5V #PWR03
 U 1 1 5257A5AA
 P 3100 1300
-F 0 "#PWR07" H 3100 1390 20  0001 C CNN
+F 0 "#PWR03" H 3100 1390 20  0001 C CNN
 F 1 "+5V" H 3100 1390 30  0000 C CNN
 F 2 "~" H 3100 1300 60  0000 C CNN
@@
 	3100 1500 3200 1500
 Connection ~ 3100 1500
-$Comp
-L AGND #PWR08
-U 1 1 5257A818
-P 3700 1600
-F 0 "#PWR08" H 3700 1600 40  0001 C CNN
-F 1 "AGND" H 3700 1530 50  0000 C CNN
-F 2 "" H 3700 1600 60  0000 C CNN
-F 3 "" H 3700 1600 60  0000 C CNN
-	1    3700 1600
-	1    0    0    -1
-$EndComp
 Wire Wire Line
 	3700 1600 3700 1500
@@
 	2400 1550 2300 1550
 Connection ~ 2400 1550
-$Comp
-L AGND #PWR09
-U 1 1 5257A963
-P 1750 1650
-F 0 "#PWR09" H 1750 1650 40  0001 C CNN
-F 1 "AGND" H 1750 1580 50  0000 C CNN
-F 2 "" H 1750 1650 60  0000 C CNN
-F 3 "" H 1750 1650 60  0000 C CNN
-	1    1750 1650
-	1    0    0    -1
-$EndComp
 Wire Wire Line
 	1750 1650 1750 1550
 Wire Wire Line
 	1750 1550 1900 1550
-$Comp
-L AGND #PWR010
-U 1 1 5257A9D6
-P 2300 4850
-F 0 "#PWR010" H 2300 4850 40  0001 C CNN
-F 1 "AGND" H 2300 4780 50  0000 C CNN
-F 2 "" H 2300 4850 60  0000 C CNN
-F 3 "" H 2300 4850 60  0000 C CNN
-	1    2300 4850
-	1    0    0    -1
-$EndComp
 Wire Wire Line
 	2300 4850 2300 4600
@@
 	3100 4600 3100 4850
 $Comp
-L AGND #PWR011
-U 1 1 5257AABC
-P 3100 4850
-F 0 "#PWR011" H 3100 4850 40  0001 C CNN
-F 1 "AGND" H 3100 4780 50  0000 C CNN
-F 2 "" H 3100 4850 60  0000 C CNN
-F 3 "" H 3100 4850 60  0000 C CNN
-	1    3100 4850
-	1    0    0    -1
-$EndComp
-$Comp
-L +5V #PWR012
+L +5V #PWR04
 U 1 1 5257AAC2
 P 2400 1300
-F 0 "#PWR012" H 2400 1390 20  0001 C CNN
+F 0 "#PWR04" H 2400 1390 20  0001 C CNN
 F 1 "+5V" H 2400 1390 30  0000 C CNN
 F 2 "~" H 2400 1300 60  0000 C CNN
@@
 $EndComp
 $Comp
-L FE_V+ #PWR013
+L FE_V+ #PWR05
 U 1 1 526E01E1
 P 6250 3850
-F 0 "#PWR013" H 6250 3950 30  0001 C CNN
+F 0 "#PWR05" H 6250 3950 30  0001 C CNN
 F 1 "FE_V+" H 6250 3950 30  0000 C CNN
 F 2 "~" H 6250 3850 60  0000 C CNN
@@
 $EndComp
 $Comp
-L FE_V+ #PWR014
+L FE_V+ #PWR06
 U 1 1 526E01F1
 P 9000 5000
-F 0 "#PWR014" H 9000 5100 30  0001 C CNN
+F 0 "#PWR06" H 9000 5100 30  0001 C CNN
 F 1 "FE_V+" H 9000 5100 30  0000 C CNN
 F 2 "~" H 9000 5000 60  0000 C CNN
@@
 $EndComp
 $Comp
-L FE_V+ #PWR015
+L FE_V+ #PWR07
 U 1 1 526E020D
 P 9000 2850
-F 0 "#PWR015" H 9000 2950 30  0001 C CNN
+F 0 "#PWR07" H 9000 2950 30  0001 C CNN
 F 1 "FE_V+" H 9000 2950 30  0000 C CNN
 F 2 "~" H 9000 2850 60  0000 C CNN
@@
 	-1   0    0    1
 $EndComp
+Wire Wire Line
+	4800 6900 4800 6800
+$Comp
+L GND_TC #PWR08
+U 1 1 5313E17A
+P 4800 6900
+F 0 "#PWR08" H 4800 6900 30  0001 C CNN
+F 1 "GND_TC" H 4800 6830 30  0000 C CNN
+F 2 "" H 4800 6900 60  0000 C CNN
+F 3 "" H 4800 6900 60  0000 C CNN
+	1    4800 6900
+	1    0    0    -1
+$EndComp
+$Comp
+L GND_TC #PWR09
+U 1 1 5313E18E
+P 3100 4850
+F 0 "#PWR09" H 3100 4850 30  0001 C CNN
+F 1 "GND_TC" H 3100 4780 30  0000 C CNN
+F 2 "" H 3100 4850 60  0000 C CNN
+F 3 "" H 3100 4850 60  0000 C CNN
+	1    3100 4850
+	1    0    0    -1
+$EndComp
+$Comp
+L GND_TC #PWR010
+U 1 1 5313E1A2
+P 2300 4850
+F 0 "#PWR010" H 2300 4850 30  0001 C CNN
+F 1 "GND_TC" H 2300 4780 30  0000 C CNN
+F 2 "" H 2300 4850 60  0000 C CNN
+F 3 "" H 2300 4850 60  0000 C CNN
+	1    2300 4850
+	1    0    0    -1
+$EndComp
+$Comp
+L GND_TC #PWR011
+U 1 1 5313E1B6
+P 4900 4700
+F 0 "#PWR011" H 4900 4700 30  0001 C CNN
+F 1 "GND_TC" H 4900 4630 30  0000 C CNN
+F 2 "" H 4900 4700 60  0000 C CNN
+F 3 "" H 4900 4700 60  0000 C CNN
+	1    4900 4700
+	1    0    0    -1
+$EndComp
+$Comp
+L GND_TC #PWR012
+U 1 1 5313E1CA
+P 5550 4000
+F 0 "#PWR012" H 5550 4000 30  0001 C CNN
+F 1 "GND_TC" H 5550 3930 30  0000 C CNN
+F 2 "" H 5550 4000 60  0000 C CNN
+F 3 "" H 5550 4000 60  0000 C CNN
+	1    5550 4000
+	1    0    0    -1
+$EndComp
+$Comp
+L GND_TC #PWR013
+U 1 1 5313E1DE
+P 5600 2800
+F 0 "#PWR013" H 5600 2800 30  0001 C CNN
+F 1 "GND_TC" H 5600 2730 30  0000 C CNN
+F 2 "" H 5600 2800 60  0000 C CNN
+F 3 "" H 5600 2800 60  0000 C CNN
+	1    5600 2800
+	1    0    0    -1
+$EndComp
+$Comp
+L GND_TC #PWR014
+U 1 1 5313E1F2
+P 1750 1650
+F 0 "#PWR014" H 1750 1650 30  0001 C CNN
+F 1 "GND_TC" H 1750 1580 30  0000 C CNN
+F 2 "" H 1750 1650 60  0000 C CNN
+F 3 "" H 1750 1650 60  0000 C CNN
+	1    1750 1650
+	1    0    0    -1
+$EndComp
+$Comp
+L GND_TC #PWR015
+U 1 1 5313E206
+P 3700 1600
+F 0 "#PWR015" H 3700 1600 30  0001 C CNN
+F 1 "GND_TC" H 3700 1530 30  0000 C CNN
+F 2 "" H 3700 1600 60  0000 C CNN
+F 3 "" H 3700 1600 60  0000 C CNN
+	1    3700 1600
+	1    0    0    -1
+$EndComp
 $EndSCHEMATC

Commit message: Layout Work Session 6
Connections:
- net GND_TC renamed AGND
Other:
- moved on the sheet: R11, R13
Changed lines of the file:
@@
 L R R11
 U 1 1 5236440B
-P 8100 2750
-F 0 "R11" V 8180 2750 40  0000 C CNN
-F 1 "R" V 8107 2751 40  0000 C CNN
-F 2 "~" V 8030 2750 30  0000 C CNN
-F 3 "~" H 8100 2750 30  0000 C CNN
-	1    8100 2750
+P 8100 2700
+F 0 "R11" V 8180 2700 40  0000 C CNN
+F 1 "R" V 8107 2701 40  0000 C CNN
+F 2 "~" V 8030 2700 30  0000 C CNN
+F 3 "~" H 8100 2700 30  0000 C CNN
+	1    8100 2700
 	1    0    0    -1
 $EndComp
@@
 L R R13
 U 1 1 5236442D
-P 8100 4000
-F 0 "R13" V 8180 4000 40  0000 C CNN
-F 1 "R" V 8107 4001 40  0000 C CNN
-F 2 "~" V 8030 4000 30  0000 C CNN
-F 3 "~" H 8100 4000 30  0000 C CNN
-	1    8100 4000
+P 8100 4075
+F 0 "R13" V 8180 4075 40  0000 C CNN
+F 1 "R" V 8107 4076 40  0000 C CNN
+F 2 "~" V 8030 4075 30  0000 C CNN
+F 3 "~" H 8100 4075 30  0000 C CNN
+	1    8100 4075
 	1    0    0    -1
 $EndComp
@@
 	7550 2350 8400 2350
 Wire Wire Line
-	8100 2350 8100 2500
-Wire Wire Line
-	8100 3000 8100 3050
-Wire Wire Line
-	8100 3700 8100 3750
-Wire Wire Line
-	8100 4250 8100 4450
+	8100 2350 8100 2450
+Wire Wire Line
+	8100 2950 8100 3050
+Wire Wire Line
+	8100 3700 8100 3825
+Wire Wire Line
+	8100 4325 8100 4450
 Wire Wire Line
 	7550 4450 8400 4450
@@
 	4800 6900 4800 6800
 $Comp
-L GND_TC #PWR08
-U 1 1 5313E17A
+L AGND #PWR08
+U 1 1 53147ADE
+P 4900 4700
+F 0 "#PWR08" H 4900 4700 40  0001 C CNN
+F 1 "AGND" H 4900 4630 50  0000 C CNN
+F 2 "" H 4900 4700 60  0000 C CNN
+F 3 "" H 4900 4700 60  0000 C CNN
+	1    4900 4700
+	1    0    0    -1
+$EndComp
+$Comp
+L AGND #PWR09
+U 1 1 53147AF2
 P 4800 6900
-F 0 "#PWR08" H 4800 6900 30  0001 C CNN
-F 1 "GND_TC" H 4800 6830 30  0000 C CNN
+F 0 "#PWR09" H 4800 6900 40  0001 C CNN
+F 1 "AGND" H 4800 6830 50  0000 C CNN
 F 2 "" H 4800 6900 60  0000 C CNN
 F 3 "" H 4800 6900 60  0000 C CNN
@@
 $EndComp
 $Comp
-L GND_TC #PWR09
-U 1 1 5313E18E
+L AGND #PWR010
+U 1 1 53147B06
+P 5550 4000
+F 0 "#PWR010" H 5550 4000 40  0001 C CNN
+F 1 "AGND" H 5550 3930 50  0000 C CNN
+F 2 "" H 5550 4000 60  0000 C CNN
+F 3 "" H 5550 4000 60  0000 C CNN
+	1    5550 4000
+	1    0    0    -1
+$EndComp
+$Comp
+L AGND #PWR011
+U 1 1 53147B1A
+P 2300 4850
+F 0 "#PWR011" H 2300 4850 40  0001 C CNN
+F 1 "AGND" H 2300 4780 50  0000 C CNN
+F 2 "" H 2300 4850 60  0000 C CNN
+F 3 "" H 2300 4850 60  0000 C CNN
+	1    2300 4850
+	1    0    0    -1
+$EndComp
+$Comp
+L AGND #PWR012
+U 1 1 53147B2C
 P 3100 4850
-F 0 "#PWR09" H 3100 4850 30  0001 C CNN
-F 1 "GND_TC" H 3100 4780 30  0000 C CNN
+F 0 "#PWR012" H 3100 4850 40  0001 C CNN
+F 1 "AGND" H 3100 4780 50  0000 C CNN
 F 2 "" H 3100 4850 60  0000 C CNN
 F 3 "" H 3100 4850 60  0000 C CNN
@@
 $EndComp
 $Comp
-L GND_TC #PWR010
-U 1 1 5313E1A2
-P 2300 4850
-F 0 "#PWR010" H 2300 4850 30  0001 C CNN
-F 1 "GND_TC" H 2300 4780 30  0000 C CNN
-F 2 "" H 2300 4850 60  0000 C CNN
-F 3 "" H 2300 4850 60  0000 C CNN
-	1    2300 4850
-	1    0    0    -1
-$EndComp
-$Comp
-L GND_TC #PWR011
-U 1 1 5313E1B6
-P 4900 4700
-F 0 "#PWR011" H 4900 4700 30  0001 C CNN
-F 1 "GND_TC" H 4900 4630 30  0000 C CNN
-F 2 "" H 4900 4700 60  0000 C CNN
-F 3 "" H 4900 4700 60  0000 C CNN
-	1    4900 4700
-	1    0    0    -1
-$EndComp
-$Comp
-L GND_TC #PWR012
-U 1 1 5313E1CA
-P 5550 4000
-F 0 "#PWR012" H 5550 4000 30  0001 C CNN
-F 1 "GND_TC" H 5550 3930 30  0000 C CNN
-F 2 "" H 5550 4000 60  0000 C CNN
-F 3 "" H 5550 4000 60  0000 C CNN
-	1    5550 4000
-	1    0    0    -1
-$EndComp
-$Comp
-L GND_TC #PWR013
-U 1 1 5313E1DE
+L AGND #PWR013
+U 1 1 53147B39
+P 1750 1650
+F 0 "#PWR013" H 1750 1650 40  0001 C CNN
+F 1 "AGND" H 1750 1580 50  0000 C CNN
+F 2 "" H 1750 1650 60  0000 C CNN
+F 3 "" H 1750 1650 60  0000 C CNN
+	1    1750 1650
+	1    0    0    -1
+$EndComp
+$Comp
+L AGND #PWR014
+U 1 1 53147B4D
+P 3700 1600
+F 0 "#PWR014" H 3700 1600 40  0001 C CNN
+F 1 "AGND" H 3700 1530 50  0000 C CNN
+F 2 "" H 3700 1600 60  0000 C CNN
+F 3 "" H 3700 1600 60  0000 C CNN
+	1    3700 1600
+	1    0    0    -1
+$EndComp
+$Comp
+L AGND #PWR015
+U 1 1 53147EB5
 P 5600 2800
-F 0 "#PWR013" H 5600 2800 30  0001 C CNN
-F 1 "GND_TC" H 5600 2730 30  0000 C CNN
+F 0 "#PWR015" H 5600 2800 40  0001 C CNN
+F 1 "AGND" H 5600 2730 50  0000 C CNN
 F 2 "" H 5600 2800 60  0000 C CNN
 F 3 "" H 5600 2800 60  0000 C CNN
@@
 	1    0    0    -1
 $EndComp
-$Comp
-L GND_TC #PWR014
-U 1 1 5313E1F2
-P 1750 1650
-F 0 "#PWR014" H 1750 1650 30  0001 C CNN
-F 1 "GND_TC" H 1750 1580 30  0000 C CNN
-F 2 "" H 1750 1650 60  0000 C CNN
-F 3 "" H 1750 1650 60  0000 C CNN
-	1    1750 1650
-	1    0    0    -1
-$EndComp
-$Comp
-L GND_TC #PWR015
-U 1 1 5313E206
-P 3700 1600
-F 0 "#PWR015" H 3700 1600 30  0001 C CNN
-F 1 "GND_TC" H 3700 1530 30  0000 C CNN
-F 2 "" H 3700 1600 60  0000 C CNN
-F 3 "" H 3700 1600 60  0000 C CNN
-	1    3700 1600
-	1    0    0    -1
-$EndComp

Commit message: Layout Work Session 6
Pulled from CE
Other:
- moved on the sheet: R11, R13
Changed lines of the file:
@@
-EESchema Schematic File Version 2
+EESchema Schematic File Version 2  date 11/10/2013 9:27:17 PM
 LIBS:power
 LIBS:device
@@
 LIBS:valves
 LIBS:BenchBuddy
-LIBS:arduino_shieldsNCL
 LIBS:BenchBuddy-cache
-EELAYER 24 0
+EELAYER 27 0
 EELAYER END
 $Descr A4 11693 8268
@@
 Sheet 2 9
 Title ""
-Date "2 nov 2013"
+Date "11 nov 2013"
 Rev ""
 Comp ""
@@
 L R R11
 U 1 1 5236440B
-P 8100 2700
-F 0 "R11" V 8180 2700 40  0000 C CNN
-F 1 "R" V 8107 2701 40  0000 C CNN
-F 2 "~" V 8030 2700 30  0000 C CNN
-F 3 "~" H 8100 2700 30  0000 C CNN
-	1    8100 2700
+P 8100 2750
+F 0 "R11" V 8180 2750 40  0000 C CNN
+F 1 "R" V 8107 2751 40  0000 C CNN
+F 2 "~" V 8030 2750 30  0000 C CNN
+F 3 "~" H 8100 2750 30  0000 C CNN
+	1    8100 2750
 	1    0    0    -1
 $EndComp
@@
 L R R13
 U 1 1 5236442D
-P 8100 4075
-F 0 "R13" V 8180 4075 40  0000 C CNN
-F 1 "R" V 8107 4076 40  0000 C CNN
-F 2 "~" V 8030 4075 30  0000 C CNN
-F 3 "~" H 8100 4075 30  0000 C CNN
-	1    8100 4075
+P 8100 4000
+F 0 "R13" V 8180 4000 40  0000 C CNN
+F 1 "R" V 8107 4001 40  0000 C CNN
+F 2 "~" V 8030 4000 30  0000 C CNN
+F 3 "~" H 8100 4000 30  0000 C CNN
+	1    8100 4000
 	1    0    0    -1
 $EndComp
@@
 	7550 2350 8400 2350
 Wire Wire Line
-	8100 2350 8100 2450
-Wire Wire Line
-	8100 2950 8100 3050
-Wire Wire Line
-	8100 3700 8100 3825
-Wire Wire Line
-	8100 4325 8100 4450
+	8100 2350 8100 2500
+Wire Wire Line
+	8100 3000 8100 3050
+Wire Wire Line
+	8100 3700 8100 3750
+Wire Wire Line
+	8100 4250 8100 4450
 Wire Wire Line
 	7550 4450 8400 4450
@@
 	5700 6800 5700 6650
 Connection ~ 5600 6800
+Wire Wire Line
+	4800 6900 4800 6800
 Connection ~ 4800 6800
 $Comp
-L +5V #PWR01
+L +5V #PWR11
 U 1 1 5257A1D1
 P 5600 5000
-F 0 "#PWR01" H 5600 5090 20  0001 C CNN
+F 0 "#PWR11" H 5600 5090 20  0001 C CNN
 F 1 "+5V" H 5600 5090 30  0000 C CNN
 F 2 "~" H 5600 5000 60  0000 C CNN
@@
 	6050 3800 6250 3800
 $Comp
-L +5V #PWR02
+L +5V #PWR12
 U 1 1 5257A5A4
 P 5600 5000
-F 0 "#PWR02" H 5600 5090 20  0001 C CNN
+F 0 "#PWR12" H 5600 5090 20  0001 C CNN
 F 1 "+5V" H 5600 5090 30  0000 C CNN
 F 2 "~" H 5600 5000 60  0000 C CNN
@@
 $EndComp
 $Comp
-L +5V #PWR03
+L +5V #PWR4
 U 1 1 5257A5AA
 P 3100 1300
-F 0 "#PWR03" H 3100 1390 20  0001 C CNN
+F 0 "#PWR4" H 3100 1390 20  0001 C CNN
 F 1 "+5V" H 3100 1390 30  0000 C CNN
 F 2 "~" H 3100 1300 60  0000 C CNN
@@
 	3100 4600 3100 4850
 $Comp
-L +5V #PWR04
+L +5V #PWR3
 U 1 1 5257AAC2
 P 2400 1300
-F 0 "#PWR04" H 2400 1390 20  0001 C CNN
+F 0 "#PWR3" H 2400 1390 20  0001 C CNN
 F 1 "+5V" H 2400 1390 30  0000 C CNN
 F 2 "~" H 2400 1300 60  0000 C CNN
@@
 $EndComp
 $Comp
-L FE_V+ #PWR05
+L FE_V+ #PWR14
 U 1 1 526E01E1
 P 6250 3850
-F 0 "#PWR05" H 6250 3950 30  0001 C CNN
+F 0 "#PWR14" H 6250 3950 30  0001 C CNN
 F 1 "FE_V+" H 6250 3950 30  0000 C CNN
 F 2 "~" H 6250 3850 60  0000 C CNN
@@
 $EndComp
 $Comp
-L FE_V+ #PWR06
+L FE_V+ #PWR18
 U 1 1 526E01F1
 P 9000 5000
-F 0 "#PWR06" H 9000 5100 30  0001 C CNN
+F 0 "#PWR18" H 9000 5100 30  0001 C CNN
 F 1 "FE_V+" H 9000 5100 30  0000 C CNN
 F 2 "~" H 9000 5000 60  0000 C CNN
@@
 $EndComp
 $Comp
-L FE_V+ #PWR07
+L FE_V+ #PWR16
 U 1 1 526E020D
 P 9000 2850
-F 0 "#PWR07" H 9000 2950 30  0001 C CNN
+F 0 "#PWR16" H 9000 2950 30  0001 C CNN
 F 1 "FE_V+" H 9000 2950 30  0000 C CNN
 F 2 "~" H 9000 2850 60  0000 C CNN
@@
 	-1   0    0    1
 $EndComp
-Wire Wire Line
-	4800 6900 4800 6800
-$Comp
-L AGND #PWR08
-U 1 1 53147ADE
+$Comp
+L AGND #PWR5
+U 1 1 527EEF67
+P 3100 4850
+F 0 "#PWR5" H 3100 4850 40  0001 C CNN
+F 1 "AGND" H 3100 4780 50  0000 C CNN
+F 2 "~" H 3100 4850 60  0000 C CNN
+F 3 "~" H 3100 4850 60  0000 C CNN
+	1    3100 4850
+	1    0    0    -1
+$EndComp
+$Comp
+L AGND #PWR2
+U 1 1 527EEF6D
+P 2300 4850
+F 0 "#PWR2" H 2300 4850 40  0001 C CNN
+F 1 "AGND" H 2300 4780 50  0000 C CNN
+F 2 "~" H 2300 4850 60  0000 C CNN
+F 3 "~" H 2300 4850 60  0000 C CNN
+	1    2300 4850
+	1    0    0    -1
+$EndComp
+$Comp
+L AGND #PWR1
+U 1 1 527EEF73
+P 1750 1650
+F 0 "#PWR1" H 1750 1650 40  0001 C CNN
+F 1 "AGND" H 1750 1580 50  0000 C CNN
+F 2 "~" H 1750 1650 60  0000 C CNN
+F 3 "~" H 1750 1650 60  0000 C CNN
+	1    1750 1650
+	1    0    0    -1
+$EndComp
+$Comp
+L AGND #PWR6
+U 1 1 527EEF79
+P 3700 1600
+F 0 "#PWR6" H 3700 1600 40  0001 C CNN
+F 1 "AGND" H 3700 1530 50  0000 C CNN
+F 2 "~" H 3700 1600 60  0000 C CNN
+F 3 "~" H 3700 1600 60  0000 C CNN
+	1    3700 1600
+	1    0    0    -1
+$EndComp
+$Comp
+L AGND #PWR10
+U 1 1 527EEF7F
+P 5600 2800
+F 0 "#PWR10" H 5600 2800 40  0001 C CNN
+F 1 "AGND" H 5600 2730 50  0000 C CNN
+F 2 "~" H 5600 2800 60  0000 C CNN
+F 3 "~" H 5600 2800 60  0000 C CNN
+	1    5600 2800
+	1    0    0    -1
+$EndComp
+$Comp
+L AGND #PWR9
+U 1 1 527EEF85
+P 5550 4000
+F 0 "#PWR9" H 5550 4000 40  0001 C CNN
+F 1 "AGND" H 5550 3930 50  0000 C CNN
+F 2 "~" H 5550 4000 60  0000 C CNN
+F 3 "~" H 5550 4000 60  0000 C CNN
+	1    5550 4000
+	1    0    0    -1
+$EndComp
+$Comp
+L AGND #PWR8
+U 1 1 527EEF8B
 P 4900 4700
-F 0 "#PWR08" H 4900 4700 40  0001 C CNN
+F 0 "#PWR8" H 4900 4700 40  0001 C CNN
 F 1 "AGND" H 4900 4630 50  0000 C CNN
-F 2 "" H 4900 4700 60  0000 C CNN
-F 3 "" H 4900 4700 60  0000 C CNN
+F 2 "~" H 4900 4700 60  0000 C CNN
+F 3 "~" H 4900 4700 60  0000 C CNN
 	1    4900 4700
 	1    0    0    -1
 $EndComp
 $Comp
-L AGND #PWR09
-U 1 1 53147AF2
+L AGND #PWR7
+U 1 1 527EEF91
 P 4800 6900
-F 0 "#PWR09" H 4800 6900 40  0001 C CNN
+F 0 "#PWR7" H 4800 6900 40  0001 C CNN
 F 1 "AGND" H 4800 6830 50  0000 C CNN
-F 2 "" H 4800 6900 60  0000 C CNN
-F 3 "" H 4800 6900 60  0000 C CNN
+F 2 "~" H 4800 6900 60  0000 C CNN
+F 3 "~" H 4800 6900 60  0000 C CNN
 	1    4800 6900
 	1    0    0    -1
 $EndComp
-$Comp
-L AGND #PWR010
-U 1 1 53147B06
-P 5550 4000
-F 0 "#PWR010" H 5550 4000 40  0001 C CNN
-F 1 "AGND" H 5550 3930 50  0000 C CNN
-F 2 "" H 5550 4000 60  0000 C CNN
-F 3 "" H 5550 4000 60  0000 C CNN
-	1    5550 4000
-	1    0    0    -1
-$EndComp
-$Comp
-L AGND #PWR011
-U 1 1 53147B1A
-P 2300 4850
-F 0 "#PWR011" H 2300 4850 40  0001 C CNN
-F 1 "AGND" H 2300 4780 50  0000 C CNN
-F 2 "" H 2300 4850 60  0000 C CNN
-F 3 "" H 2300 4850 60  0000 C CNN
-	1    2300 4850
-	1    0    0    -1
-$EndComp
-$Comp
-L AGND #PWR012
-U 1 1 53147B2C
-P 3100 4850
-F 0 "#PWR012" H 3100 4850 40  0001 C CNN
-F 1 "AGND" H 3100 4780 50  0000 C CNN
-F 2 "" H 3100 4850 60  0000 C CNN
-F 3 "" H 3100 4850 60  0000 C CNN
-	1    3100 4850
-	1    0    0    -1
-$EndComp
-$Comp
-L AGND #PWR013
-U 1 1 53147B39
-P 1750 1650
-F 0 "#PWR013" H 1750 1650 40  0001 C CNN
-F 1 "AGND" H 1750 1580 50  0000 C CNN
-F 2 "" H 1750 1650 60  0000 C CNN
-F 3 "" H 1750 1650 60  0000 C CNN
-	1    1750 1650
-	1    0    0    -1
-$EndComp
-$Comp
-L AGND #PWR014
-U 1 1 53147B4D
-P 3700 1600
-F 0 "#PWR014" H 3700 1600 40  0001 C CNN
-F 1 "AGND" H 3700 1530 50  0000 C CNN
-F 2 "" H 3700 1600 60  0000 C CNN
-F 3 "" H 3700 1600 60  0000 C CNN
-	1    3700 1600
-	1    0    0    -1
-$EndComp
-$Comp
-L AGND #PWR015
-U 1 1 53147EB5
-P 5600 2800
-F 0 "#PWR015" H 5600 2800 40  0001 C CNN
-F 1 "AGND" H 5600 2730 50  0000 C CNN
-F 2 "" H 5600 2800 60  0000 C CNN
-F 3 "" H 5600 2800 60  0000 C CNN
-	1    5600 2800
-	1    0    0    -1
-$EndComp
