File: _autosave-BenchBuddy.kicad_pcb (KiCad board)
At the start: 4 copper layers, 165.1 x 63.5 mm, 133 parts, among them K1 1461069-5, P1 24 Pin MiniFit JR, P2 CONN_3X2, P3 CONN_2, P4 12 Pin Terminal Block, P5 3 Pin TB, Q1 2N3904, Q2 DMN65D8L-7, Q3 AOD476, Q4 AOD476, SW1 Power Switch, U1 LTV-816S, U11 LM317, U2 MCP3901, U3 LMT84, U4 OPA4170, U5 MCP4801, U6 LM337T, U7 AP5726, U8 LM337T, U9 LM317

Commit message: Layout Work Session 7
Pulled from CE
Parts:
- R12, R44, R45, U3: moved to F.Cu
- moved P2 25.5 mm to (179.8, 96.6)
- moved D4 17.4 mm to (205.5, 103.6)
- moved R44 14.9 mm to (186.2, 93.8), turned to 0 degrees
- moved R45 13.6 mm to (186.1, 98.6), turned to 0 degrees
- moved R12 13.5 mm to (186.2, 96.2), turned to 0 degrees
- moved R10 6.88 mm to (188.7, 97.8)
- moved U4 5.00 mm to (194.6, 98.0)
- moved R11 3.56 mm to (202.1, 97.5), turned to 270 degrees
- moved C9 3.05 mm to (191.7, 94.8)
- moved R9 3.05 mm to (198.1, 98.0)
- moved R13 3.05 mm to (192.2, 99.0)
- moved C15 2.88 mm to (210.0, 89.5), turned to 90 degrees
- moved C25 2.80 mm to (200.2, 91.9)
- moved U3 1.82 mm to (210.4, 97.0), turned to 90 degrees
- moved Q4 1.65 mm to (187.3, 108.1)
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Connections:
- P4 pad 8: +5P -> +5V
Routing:
- net -12V: track 212.4 -> 205.8 mm, vias 2 -> 1
- net +12V: track 209.0 -> 203.4 mm
- net AGND: track 0.00 -> 1.91 mm, vias 0 -> 1
- net +5V: track 8.35 -> 7.83 mm
- removed copper zone on F.Cu, net /Arduino/CURR_MEAS
- removed copper zone on F.Cu, net /Fan/FAN_OUT-
