File: Power.sch (KiCad schematic (older format))
At the start: 18 parts, among them P1 24 Pin MiniFit JR, SW1 Power Switch

Commit message: Layout Work Session 8
Parts:
- removed JP1, JP2, JP3, JP4: JUMPER, ~, symbol JUMPER
- removed TP1: CONN_1, symbol CONN_1
- added SP1: PWR_STAR_POINT, symbol PWR_STAR_POINT
Connections:
- wire segments 63 -> 57

Commit message: Layout Work Session 12
Pulled from CE.

Session 11 missed due to corrupted pcb file pulled from CE
Parts:
- removed SP1: PWR_STAR_POINT, symbol PWR_STAR_POINT
- added JP1, JP2, JP3, JP4: JUMPER, ~, symbol JUMPER
- added TP1: CONN_1, symbol CONN_1
Connections:
- wire segments 57 -> 61
